File: pcbs/tulip4_board/tulip breakout.brd (EAGLE design)
At the start: 86.3 x 47.6 mm, 50 parts, among them IC1 CP2102N-A02-GQFN24, U1 ESP32-S3-WROOM-2-N32R8V, U2 6N138SDM, U4 UDA1334ATS, X2 FH12-40S-0.5SH, X3 19269, X5 19269, X6 19269

Commit message: .
Parts:
- added IC2: LM2937, linear:TO263-3
Connections:
- removed net 5V: CONNHEADER.8, U2.8, USB_KEYBOARD.1, X2.39, X2.40
- net 3V3: now also IC2.3
- net 5V_USB: now also CONNHEADER.8, IC2.1, U2.8, USB_KEYBOARD.1, X2.39, X2.40
- net GND: now also IC2.2
Routing:
- net 5V_USB: track 36.7 -> 190.7 mm, vias 4 -> 11
- net 5V: track 90.5 -> 0.00 mm, vias 5 -> 0
- net 3V3: track 195.0 -> 240.4 mm, vias 6 -> 8
- net GND: track 357.0 -> 362.7 mm
Changed lines of the file:
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@@
 <attribute name="VALUE" x="20.932" y="20.738" size="0.4064" layer="27" ratio="10"/>
+</element>
+<element name="IC2" library="linear" library_urn="urn:adsk.eagle:library:262" package="TO263-3" package3d_urn="urn:adsk.eagle:package:16425/2" value="LM2937" x="90.1" y="40.6" smashed="yes">
+<attribute name="NAME" x="84.512" y="35.012" size="1.27" layer="25" rot="R90"/>
+<attribute name="POPULARITY" value="0" x="90.1" y="40.6" size="1.778" layer="27" display="off"/>
+<attribute name="VALUE" x="96.958" y="35.012" size="1.27" layer="27" rot="R90"/>
 </element>
 </elements>
@@
 <via x="38.625" y="44.125" extent="1-16" drill="0.254"/>
 <via x="15.25" y="42.75" extent="1-16" drill="0.254"/>
-</signal>
-<signal name="5V">
-<contactref element="USB_KEYBOARD" pad="1"/>
-<contactref element="X2" pad="39"/>
-<contactref element="X2" pad="40"/>
-<contactref element="CONNHEADER" pad="8"/>
-<contactref element="U2" pad="8"/>
-<wire x1="40.375" y1="38" x2="40" y2="38" width="0.1524" layer="1"/>
-<wire x1="40" y1="38" x2="39.95" y2="38.05" width="0.1524" layer="1"/>
-<wire x1="40.375" y1="38" x2="40.45" y2="38.05" width="0.1524" layer="1"/>
-<wire x1="40.375" y1="39.125" x2="40.375" y2="38.125" width="0.1524" layer="1"/>
-<wire x1="40.25" y1="39.125" x2="40.375" y2="39.125" width="0.1524" layer="1"/>
-<wire x1="43.125" y1="36.25" x2="40.25" y2="39.125" width="0.1524" layer="16"/>
-<wire x1="43.25" y1="36.125" x2="43.125" y2="36.25" width="0.1524" layer="1"/>
-<wire x1="49.625" y1="36.125" x2="43.25" y2="36.125" width="0.1524" layer="1"/>
-<wire x1="50.875" y1="34.875" x2="49.625" y2="36.125" width="0.1524" layer="1"/>
-<wire x1="40.375" y1="38.125" x2="40.45" y2="38.05" width="0.1524" layer="1"/>
-<wire x1="50.875" y1="34.875" x2="50.97" y2="34.77" width="0.1524" layer="1"/>
-<wire x1="81.75" y1="41.25" x2="82.625" y2="42.125" width="0.1524" layer="1"/>
-<wire x1="74.75" y1="41.25" x2="81.75" y2="41.25" width="0.1524" layer="1"/>
-<wire x1="74.5" y1="41" x2="74.75" y2="41.25" width="0.1524" layer="1"/>
-<wire x1="62.75" y1="41" x2="74.5" y2="41" width="0.1524" layer="1"/>
-<wire x1="57.75" y1="41" x2="62.75" y2="41" width="0.1524" layer="16"/>
-<wire x1="57.75" y1="38.875" x2="57.75" y2="41" width="0.1524" layer="16"/>
-<wire x1="57.125" y1="38.25" x2="57.75" y2="38.875" width="0.1524" layer="16"/>
-<wire x1="51" y1="38.25" x2="57.125" y2="38.25" width="0.1524" layer="16"/>
-<wire x1="51" y1="34.875" x2="51" y2="38.25" width="0.1524" layer="16"/>
-<wire x1="82.625" y1="42.125" x2="82.705" y2="42.21" width="0.1524" layer="1"/>
-<wire x1="51" y1="34.875" x2="50.97" y2="34.77" width="0.1524" layer="16"/>
-<wire x1="14.75" y1="37" x2="12.875" y2="35.125" width="0.1524" layer="16"/>
-<wire x1="14.75" y1="43" x2="14.75" y2="37" width="0.1524" layer="16"/>
-<wire x1="15.375" y1="43.625" x2="14.75" y2="43" width="0.1524" layer="16"/>
-<wire x1="22.375" y1="43.625" x2="15.375" y2="43.625" width="0.1524" layer="16"/>
-<wire x1="33.75" y1="43.625" x2="22.375" y2="43.625" width="0.1524" layer="1"/>
-<wire x1="38.625" y1="43.625" x2="33.75" y2="43.625" width="0.1524" layer="16"/>
-<wire x1="40.25" y1="42" x2="38.625" y2="43.625" width="0.1524" layer="16"/>
-<wire x1="40.25" y1="39.125" x2="40.25" y2="42" width="0.1524" layer="16"/>
-<wire x1="12.875" y1="35.125" x2="12.82" y2="35.01" width="0.1524" layer="16"/>
-<via x="40.25" y="39.125" extent="1-16" drill="0.254"/>
-<via x="43.125" y="36.25" extent="1-16" drill="0.254"/>
-<via x="62.75" y="41" extent="1-16" drill="0.254"/>
-<via x="22.375" y="43.625" extent="1-16" drill="0.254"/>
-<via x="33.75" y="43.625" extent="1-16" drill="0.254"/>
+<contactref element="IC2" pad="2"/>
+<wire x1="90" y1="31" x2="90" y2="34.5" width="0.1524" layer="1"/>
+<wire x1="88.5" y1="31" x2="90" y2="31" width="0.1524" layer="1"/>
+<wire x1="90" y1="34.5" x2="90.1" y2="34.8088" width="0.1524" layer="1"/>
+<wire x1="88.5" y1="31" x2="88.3" y2="30.8" width="0.1524" layer="1"/>
 </signal>
 <signal name="MIDI_IN_SOURCE">
@@
 <via x="17.75" y="6.875" extent="1-16" drill="0.254"/>
 <via x="48.875" y="14.25" extent="1-16" drill="0.254"/>
+<contactref element="IC2" pad="3"/>
+<wire x1="91.5" y1="34.5" x2="92.5" y2="34.5" width="0.1524" layer="1"/>
+<wire x1="70" y1="34.5" x2="91.5" y2="34.5" width="0.1524" layer="16"/>
+<wire x1="70" y1="16" x2="70" y2="34.5" width="0.1524" layer="16"/>
+<wire x1="69" y1="15" x2="70" y2="16" width="0.1524" layer="1"/>
+<wire x1="67.5" y1="15" x2="69" y2="15" width="0.1524" layer="1"/>
+<wire x1="67.5" y1="14" x2="67.5" y2="15" width="0.1524" layer="1"/>
+<wire x1="92.5" y1="34.5" x2="92.64" y2="34.8088" width="0.1524" layer="1"/>
+<wire x1="67.5" y1="14" x2="67.475" y2="13.88" width="0.1524" layer="1"/>
+<via x="91.5" y="34.5" extent="1-16" drill="0.254"/>
+<via x="70" y="16" extent="1-16" drill="0.254"/>
 </signal>
 <signal name="INT">
@@
 <via x="23.5" y="15.625" extent="1-16" drill="0.254"/>
 <via x="28.875" y="10.25" extent="1-16" drill="0.254"/>
+<contactref element="IC2" pad="1"/>
+<contactref element="USB_KEYBOARD" pad="1"/>
+<contactref element="X2" pad="39"/>
+<contactref element="X2" pad="40"/>
+<contactref element="CONNHEADER" pad="8"/>
+<contactref element="U2" pad="8"/>
+<wire x1="40.375" y1="38" x2="40" y2="38" width="0.1524" layer="1"/>
+<wire x1="40" y1="38" x2="39.95" y2="38.05" width="0.1524" layer="1"/>
+<wire x1="40.375" y1="38" x2="40.45" y2="38.05" width="0.1524" layer="1"/>
+<wire x1="40.375" y1="39.125" x2="40.375" y2="38.125" width="0.1524" layer="1"/>
+<wire x1="40.25" y1="39.125" x2="40.375" y2="39.125" width="0.1524" layer="1"/>
+<wire x1="43.125" y1="36.25" x2="40.25" y2="39.125" width="0.1524" layer="16"/>
+<wire x1="43.25" y1="36.125" x2="43.125" y2="36.25" width="0.1524" layer="1"/>
+<wire x1="49.625" y1="36.125" x2="43.25" y2="36.125" width="0.1524" layer="1"/>
+<wire x1="50.875" y1="34.875" x2="49.625" y2="36.125" width="0.1524" layer="1"/>
+<wire x1="40.375" y1="38.125" x2="40.45" y2="38.05" width="0.1524" layer="1"/>
+<wire x1="50.875" y1="34.875" x2="50.97" y2="34.77" width="0.1524" layer="1"/>
+<wire x1="81.75" y1="41.25" x2="82.625" y2="42.125" width="0.1524" layer="1"/>
+<wire x1="74.75" y1="41.25" x2="81.75" y2="41.25" width="0.1524" layer="1"/>
+<wire x1="74.5" y1="41" x2="74.75" y2="41.25" width="0.1524" layer="1"/>
+<wire x1="62.75" y1="41" x2="74.5" y2="41" width="0.1524" layer="1"/>
+<wire x1="57.75" y1="41" x2="61" y2="41" width="0.1524" layer="16"/>
+<wire x1="61" y1="41" x2="62.75" y2="41" width="0.1524" layer="16"/>
+<wire x1="57.75" y1="38.875" x2="57.75" y2="41" width="0.1524" layer="16"/>
+<wire x1="57.125" y1="38.25" x2="57.75" y2="38.875" width="0.1524" layer="16"/>
+<wire x1="51" y1="38.25" x2="57.125" y2="38.25" width="0.1524" layer="16"/>
+<wire x1="51" y1="34.875" x2="51" y2="38.25" width="0.1524" layer="16"/>
+<wire x1="82.625" y1="42.125" x2="82.705" y2="42.21" width="0.1524" layer="1"/>
+<wire x1="51" y1="34.875" x2="50.97" y2="34.77" width="0.1524" layer="16"/>
+<wire x1="14.75" y1="37" x2="12.875" y2="35.125" width="0.1524" layer="16"/>
+<wire x1="14.75" y1="43" x2="14.75" y2="37" width="0.1524" layer="16"/>
+<wire x1="15.375" y1="43.625" x2="14.75" y2="43" width="0.1524" layer="16"/>
+<wire x1="22.375" y1="43.625" x2="15.375" y2="43.625" width="0.1524" layer="16"/>
+<wire x1="33.75" y1="43.625" x2="22.375" y2="43.625" width="0.1524" layer="1"/>
+<wire x1="38.625" y1="43.625" x2="33.75" y2="43.625" width="0.1524" layer="16"/>
+<wire x1="40.25" y1="42" x2="38.625" y2="43.625" width="0.1524" layer="16"/>
+<wire x1="40.25" y1="39.125" x2="40.25" y2="42" width="0.1524" layer="16"/>
+<wire x1="12.875" y1="35.125" x2="12.82" y2="35.01" width="0.1524" layer="16"/>
+<via x="40.25" y="39.125" extent="1-16" drill="0.254"/>
+<via x="43.125" y="36.25" extent="1-16" drill="0.254"/>
+<via x="62.75" y="41" extent="1-16" drill="0.254"/>
+<via x="22.375" y="43.625" extent="1-16" drill="0.254"/>
+<via x="33.75" y="43.625" extent="1-16" drill="0.254"/>
+<wire x1="84" y1="35" x2="87.5" y2="35" width="0.1524" layer="1"/>
+<wire x1="69" y1="35" x2="84" y2="35" width="0.1524" layer="16"/>
+<wire x1="69" y1="37.5" x2="69" y2="35" width="0.1524" layer="16"/>
+<wire x1="62" y1="44.5" x2="69" y2="37.5" width="0.1524" layer="16"/>
+<wire x1="61" y1="44.5" x2="62" y2="44.5" width="0.1524" layer="16"/>
+<wire x1="61" y1="41" x2="61" y2="44.5" width="0.1524" layer="16"/>
+<wire x1="87.5" y1="35" x2="87.56" y2="34.8088" width="0.1524" layer="1"/>
+<wire x1="19.5" y1="16" x2="20.5" y2="17" width="0.1524" layer="1"/>
+<wire x1="14.5" y1="16" x2="19.5" y2="16" width="0.1524" layer="1"/>
+<wire x1="11.5" y1="19" x2="14.5" y2="16" width="0.1524" layer="16"/>
+<wire x1="11.5" y1="27" x2="11.5" y2="19" width="0.1524" layer="16"/>
+<wire x1="11" y1="27.5" x2="11.5" y2="27" width="0.1524" layer="16"/>
+<wire x1="11" y1="33.5" x2="11" y2="27.5" width="0.1524" layer="16"/>
+<wire x1="12.5" y1="35" x2="11" y2="33.5" width="0.1524" layer="16"/>
+<wire x1="20.5" y1="17" x2="20.65" y2="17" width="0.1524" layer="1"/>
+<wire x1="12.5" y1="35" x2="12.82" y2="35.01" width="0.1524" layer="16"/>
+<via x="84" y="35" extent="1-16" drill="0.254"/>
+<via x="14.5" y="16" extent="1-16" drill="0.254"/>
 </signal>
 <signal name="!RTS">

Commit message: .
Parts:
- removed IC1: CP2102N-A02-GQFN24, CP2102N-A02-GQFN24:QFN50P400X400X80-25N
- removed IC2: LM2937, linear:TO263-3
- removed U$6: MBT3904DW1T1G, MBT3904DW1T1G:SOT236
- removed U2: 6N138SDM, 6N138SDM:COUPL_6N138SDM
- removed U4: UDA1334ATS, microbuilder:SSOP16_4.4MM
- removed USB_KEYBOARD: (no value), con-berg:PN87520
- removed X1: (no value), microbuilder:USB_C_CUSB31-CFM2AX-01-X
- removed X3, X5, X6: 19269, microbuilder:4UCONN_19269
- added 6N138: 6N138SDM, 6N138SDM:COUPL_6N138SDM
- added AUDIO_CONN, MIDI_IN_CONN, MIDI_OUT_CONN: 19269, microbuilder:4UCONN_19269
- added CP2102: CP2102N-A02-GQFN24, CP2102N-A02-GQFN24:QFN50P400X400X80-25N
- added J1: CSP-USC16-TR, CSP-USC16-TR:VALCON_CSP-USC16-TR
- added REG: TS1117BCW33_RPG, TS1117BCW33_RPG:VREG_TS1117BCW33_RPG
- added RESET: MBT3904DW1T1G, MBT3904DW1T1G:SOT236
- added UDA1334: UDA1334ATS, microbuilder:SSOP16_4.4MM
- added USBKB: USB-A-S-X-X-SM2, USB-A-S-X-X-SM2:SAMTEC_USB-A-S-X-X-SM2
- R1, R10, R11, R12, R13, R14, R15, R16, R17, R18, R5, R6, R7: device microbuilder:0603-NO -> adafruit:R0805
- R2, R22, R23, R3, R4, R8, R9: device microbuilder:0805-NO -> adafruit:R0805
- moved FB4 53.6 mm to (73.1, 12.9)
- moved FB3 48.9 mm to (73.0, 8.90)
- moved C4 47.4 mm to (15.8, 37.4), turned to 90 degrees
- moved R12 44.9 mm to (75.1, 43.9)
- moved R16 42.0 mm to (75.0, 41.0)
- moved R1 38.6 mm to (23.1, 4.90), turned to 180 degrees
- moved C12 35.4 mm to (52.7, 14.1)
- moved R18 35.2 mm to (75.0, 35.0)
- moved R17 35.0 mm to (75.0, 38.0)
- moved R14 33.2 mm to (22.0, 22.9)
- moved R10 30.3 mm to (43.0, 26.0)
- moved C14 29.6 mm to (64.6, 11.2)
- moved R5 29.5 mm to (18.0, 8.90), turned to 180 degrees
- moved R7 27.8 mm to (18.0, 4.90), turned to 180 degrees
- moved R15 24.5 mm to (67.1, 43.8)
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Connections:
- removed net CC1: R11.2, X1.A5
- removed net CC2: R10.2, X1.B5
- new net N$3: J1.B5, R11.2
- new net N$4: J1.A5, R10.2
- net !DTR: now also CP2102.23, RESET.4; no longer IC1.23, U$6.4
- net !RTS: now also CP2102.19, RESET.1; no longer IC1.19, U$6.1
- net 3V3: now also REG.2, REG.4, UDA1334.4; no longer IC2.3, U4.4
- net 3V3_USB: now also CP2102.5, CP2102.6; no longer IC1.5, IC1.6
- net 5V_USB: now also 6N138.8, CP2102.7, J1.A4, J1.A9, J1.B4, J1.B9, REG.3, USBKB.01; no longer IC1.7, IC2.1, U2.8, USB_KEYBOARD.1, X1.A4B9, X1.B4A9
- net AGND: now also AUDIO_CONN.1, UDA1334.15; no longer U4.15, X6.1
- net BCLK: now also UDA1334.1; no longer U4.1
- net D+: now also USBKB.03; no longer USB_KEYBOARD.3
- net D-: now also USBKB.02; no longer USB_KEYBOARD.2
- net DIN: now also UDA1334.3; no longer U4.3
- net ESP32_EN: now also RESET.6; no longer U$6.6
- net GND: now also 6N138.5, CP2102.2, CP2102.25, J1.A1, J1.A12, J1.B1, J1.B12, J1.S1, J1.S2, J1.S3, J1.S4, MIDI_IN_CONN.1, MIDI_OUT_CONN.1, REG.1, UDA1334.10, UDA1334.11, UDA1334.5, UDA1334.6, UDA1334.7, UDA1334.8, UDA1334.9, USBKB.04, USBKB.S1, USBKB.S2; no longer IC1.2, IC1.25, IC2.2, U2.5, U4.10, U4.11, U4.5, U4.6, U4.7, U4.8, U4.9, USB_KEYBOARD.4, X1.A1B12, X1.B1A12, X3.1, X5.1
- net IO0: now also RESET.3; no longer U$6.3
- net LOUT: now also AUDIO_CONN.2, AUDIO_CONN.4; no longer X6.2, X6.4
- net LRC: now also UDA1334.2; no longer U4.2
- net MIDI_IN: now also 6N138.6; no longer U2.6
- net MIDI_IN_SINK: now also 6N138.3, MIDI_IN_CONN.2, MIDI_IN_CONN.4; no longer U2.3, X5.2, X5.4
- net MIDI_IN_SOURCE: now also MIDI_IN_CONN.3, MIDI_IN_CONN.5; no longer X5.3, X5.5
- net MIDI_OUT_SINK: now also MIDI_OUT_CONN.2, MIDI_OUT_CONN.4; no longer X3.2, X3.4
- net MIDI_OUT_SOURCE: now also MIDI_OUT_CONN.3, MIDI_OUT_CONN.5; no longer X3.3, X3.5
- net N$1: now also RESET.2; no longer U$6.2
- net N$10: now also UDA1334.12; no longer U4.12
- net N$11: now also UDA1334.16; no longer U4.16
- net N$12: now also UDA1334.14; no longer U4.14
- net N$2: now also RESET.5; no longer U$6.5
- net N$30: now also 6N138.2; no longer U2.2
- net N$32: now also 6N138.7; no longer U2.7
- net N$5: now also UDA1334.13; no longer U4.13
- net ROUT: now also AUDIO_CONN.3, AUDIO_CONN.5; no longer X6.3, X6.5
- net UART0_RXD: now also CP2102.21; no longer IC1.21
- net UART0_TXD: now also CP2102.20; no longer IC1.20
- net USBC_D+: now also CP2102.3, J1.A6; no longer IC1.3, X1.A6, X1.B6
- net USBC_D-: now also CP2102.4, J1.A7; no longer IC1.4, X1.A7, X1.B7
- net USB_RESET: now also CP2102.9; no longer IC1.9
- net USB_VBUS: now also CP2102.8; no longer IC1.8
Routing:
- net D+: track 5.61 -> 75.7 mm, vias 0 -> 2
- net AGND: track 137.1 -> 76.1 mm, vias 5 -> 1
- net N$4: track 0.00 -> 52.7 mm, vias 0 -> 2
- net 3V3: track 240.4 -> 190.3 mm, vias 8 -> 9
- net N$1: track 68.5 -> 24.3 mm, vias 0 -> 2
- net N$32: track 60.8 -> 17.5 mm, vias 2 -> 0
- net N$10: track 60.6 -> 17.7 mm
- net D-: track 5.91 -> 45.8 mm, vias 0 -> 2
- net !DTR: track 69.5 -> 30.8 mm
- net SCL: track 96.9 -> 59.5 mm, vias 4 -> 7
- net DIN: track 60.5 -> 96.5 mm
- net N$5: track 68.1 -> 40.3 mm, vias 5 -> 3
- net ROUT: track 87.5 -> 60.2 mm
- net MIDI_IN_SINK: track 64.1 -> 88.1 mm
- net N$3: track 0.00 -> 23.2 mm, vias 0 -> 2
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Other:
- board size 86.3 x 47.6 mm -> 81.1 x 46 mm
- board text added: "tulip.computer v4/r0"

Commit message: .
Parts:
- removed 6N138: 6N138SDM, 6N138SDM:COUPL_6N138SDM
- removed C11, C12, C15: 0.1uF, microbuilder:0805-NO
- removed C13, C14: 0.01uF, microbuilder:0805-NO
- removed C16, C17: 47uF, microbuilder:PANASONIC_C
- removed C18, C19, C20: 10uF, microbuilder:0805-NO
- removed CP2102: CP2102N-A02-GQFN24, CP2102N-A02-GQFN24:QFN50P400X400X80-25N
- removed FB3, FB4: Ferrite, microbuilder:0805
- removed R22, R8: 220k, adafruit:R0805
- removed R23, R9: 100, adafruit:R0805
- removed R4: 10k, adafruit:R0805
- removed REG: TS1117BCW33_RPG, TS1117BCW33_RPG:VREG_TS1117BCW33_RPG
- removed UDA1334: UDA1334ATS, microbuilder:SSOP16_4.4MM
- added 6N137S: 6N137S, 6N137S:8-SMD
- added C10, C21, C8, C9: 0.1uF, microbuilder:0805-NO
- added C22, C23: 2.2uF, microbuilder:0805-NO
- added C28, C29, C30, C31: 10uF, microbuilder:PANASONIC_C
- added C32, C33: 2.2nF, microbuilder:0805-NO
- added R19, R20: 470, adafruit:R0805
- added U2: INTERFACE-CP2102-GMR(QFN28), INTERFACE-CP2102-GMR_QFN28_:QFN28G_0.5-5X5MM
- added U3: PCM5101APW, pcm5101apw:PW20_TEX
Connections:
- removed net N$10: C15.1, C20.1, UDA1334.12
- removed net N$11: C17.+, UDA1334.16
- removed net N$12: C16.+, UDA1334.14
- removed net N$5: C11.1, C18.1, FB3.1, UDA1334.13
- removed net N$6: C16.-, R8.2, R9.1
- removed net N$9: C17.-, R22.2, R23.1
- removed net USB_RESET: CP2102.9, R4.1
- new net N$16: C22.1, U3.4
- new net N$18: C22.2, U3.2
- new net N$7: C28.+, C8.1, U3.18
- new net N$8: R19.2, U3.7
- new net OUTL: R20.2, U3.6
- new net VNEG: C23.1, U3.5
- net !DTR: now also U2.28; no longer CP2102.23
- net !RTS: now also U2.24; no longer CP2102.19
- net 3V3: now also C10.2, C21.2, C29.+, C30.+, C31.+, C9.2, U2.6, U3.1, U3.17, U3.20, U3.8; no longer C12.1, C19.1, FB3.2, REG.2, REG.4, UDA1334.4
- net 3V3_USB: no longer CP2102.5, CP2102.6, R4.2
- net 5V_USB: now also 6N137S.8, U2.7; no longer 6N138.8, CP2102.7, REG.3
- net AGND: now also C21.1, C23.2, C30.-, C31.-, C32.2, C33.2, C9.1, U3.3, U3.9; no longer C11.2, C13.2, C14.2, C15.2, C18.2, C20.2, FB4.1, R22.1, R8.1, UDA1334.15
- net BCLK: now also U3.13; no longer UDA1334.1
- net DIN: now also U3.14; no longer UDA1334.3
- net GND: now also 6N137S.5, C10.1, C28.-, C29.-, C8.2, U2.29, U2.3, U3.10, U3.11, U3.12, U3.16, U3.19; no longer 6N138.5, C12.2, C19.2, CP2102.2, CP2102.25, FB4.2, REG.1, UDA1334.10, UDA1334.11, UDA1334.5, UDA1334.6, UDA1334.7, UDA1334.8, UDA1334.9
- net LOUT: now also C33.1, R20.1; no longer C13.1, R9.2
- net LRC: now also U3.15; no longer UDA1334.2
- net MIDI_IN: now also 6N137S.6; no longer 6N138.6
- net MIDI_IN_SINK: now also 6N137S.3; no longer 6N138.3
- net N$30: now also 6N137S.2; no longer 6N138.2
- net N$32: now also 6N137S.7; no longer 6N138.7
- net ROUT: now also C32.1, R19.1; no longer C14.1, R23.2
- net UART0_RXD: now also U2.26; no longer CP2102.21
- net UART0_TXD: now also U2.25; no longer CP2102.20
- net USBC_D+: now also U2.4; no longer CP2102.3
- net USBC_D-: now also U2.5; no longer CP2102.4
- net USB_VBUS: now also U2.8; no longer CP2102.8
Routing:
- net 3V3: track 190.3 -> 241.3 mm, vias 9 -> 8
- net PWR: track 37.7 -> 85.0 mm
- net N$6: track 43.9 -> 0.00 mm, vias 2 -> 0
- net N$5: track 40.3 -> 0.00 mm, vias 3 -> 0
- net 3V3_USB: track 46.3 -> 6.59 mm, vias 3 -> 0
- net DIN: track 96.5 -> 57.4 mm, vias 2 -> 4
- net USB_RESET: track 34.9 -> 0.00 mm, vias 2 -> 0
- net N$7: track 0.00 -> 33.3 mm, vias 0 -> 2
- net MIDI_IN_SINK: track 88.1 -> 55.3 mm, vias 2 -> 4
- net AGND: track 76.1 -> 106.0 mm, vias 1 -> 2
- net N$16: track 0.00 -> 29.8 mm
- net N$30: track 57.5 -> 33.2 mm
- net OUTL: track 0.00 -> 23.2 mm
- net N$9: track 22.9 -> 0.00 mm, vias 2 -> 0
- net D+: track 75.7 -> 54.6 mm
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
Commit message: .
Parts:
- added R4: 10k, adafruit:R0805
- moved C23 4.10 mm to (61.6, 13.2)
- moved C9 4.10 mm to (61.6, 19.1)
- moved C33 4.00 mm to (61.6, 10.1)
- moved C21 4.00 mm to (61.6, 16.1)
- moved U2 3.11 mm to (29.8, 14.9)
- moved C32 2.91 mm to (55.7, 10.1)
- moved C10 2.90 mm to (55.6, 16.1)
- moved C8 2.90 mm to (55.7, 19.2)
- moved USBKB 2.81 mm to (49.6, 2.40)
- moved C22 2.80 mm to (55.7, 13.2)
- moved U3 2.30 mm to (71.9, 19.4)
- moved J1 2.24 mm to (33.1, 7.50)
- moved R19 1.90 mm to (50.1, 19.0)
- moved R20 1.90 mm to (50.1, 16.0)
- moved D2 0.58 mm to (74.8, 29.9), turned to 90 degrees
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Connections:
- removed net 3V3_USB: C2.1, C3.1
- new net USB_RESET: R4.1, U2.9
- net 3V3: now also C2.1, C3.1, R4.2
Routing:
- net PWR: track 85.0 -> 44.2 mm, vias 1 -> 2
- net MIDI_IN: track 80.6 -> 117.1 mm, vias 2 -> 4
- net R7: track 36.8 -> 72.2 mm
- net 3V3: track 241.3 -> 268.0 mm
- net N$2: track 23.8 -> 49.8 mm, vias 2 -> 0
- net MIDI_IN_SINK: track 55.3 -> 80.0 mm, vias 4 -> 2
- net LRC: track 84.3 -> 106.8 mm, vias 4 -> 2
- net MIDI_OUT_SINK: track 49.4 -> 70.1 mm, vias 4 -> 0
- net AGND: track 106.0 -> 85.4 mm
- net MIDI_OUT: track 57.8 -> 78.1 mm
- net 5V_USB: track 161.5 -> 178.2 mm, vias 5 -> 4
- net N$32: track 17.3 -> 32.0 mm
- net USB_RESET: track 0.00 -> 14.0 mm, vias 0 -> 2
- net B6: track 38.8 -> 52.5 mm
- net N$16: track 29.8 -> 18.3 mm, vias 0 -> 2
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