File: pcbs/tulip4_board/tulip breakout.sch (EAGLE design)
At the start: 50 parts, among them IC1 CP2102N-A02-GQFN24, U1 ESP32-S3-WROOM-2-N32R8V, U2 6N138SDM, U4 UDA1334ATS, X2 FH12-40S-0.5SH, X3 19269, X5 19269, X6 19269

Commit message: .
Parts:
- added IC2: LM2937, linear:LM2937
Connections:
- removed net 5V: CONNHEADER.8, U2.VCC, USB_KEYBOARD.1, X2-39.1, X2-40.1
- net 3V3: now also IC2.VO
- net 5V_USB: now also CONNHEADER.8, IC2.VI, U2.VCC, USB_KEYBOARD.1, X2-39.1, X2-40.1
- net GND: now also IC2.GND
Changed lines of the file:
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@@
 <grid distance="0.1" unitdist="inch" unit="inch" style="lines" multiple="1" display="no" altdistance="0.01" altunitdist="inch" altunit="inch"/>
 <layers>
-<layer number="1" name="Top" color="4" fill="1" visible="yes" active="no"/>
-<layer number="16" name="Bottom" color="1" fill="1" visible="yes" active="no"/>
-<layer number="17" name="Pads" color="2" fill="1" visible="yes" active="no"/>
-<layer number="18" name="Vias" color="2" fill="1" visible="yes" active="no"/>
-<layer number="19" name="Unrouted" color="6" fill="1" visible="yes" active="no"/>
-<layer number="20" name="Dimension" color="24" fill="1" visible="yes" active="no"/>
-<layer number="21" name="tPlace" color="7" fill="1" visible="yes" active="no"/>
-<layer number="22" name="bPlace" color="7" fill="1" visible="yes" active="no"/>
-<layer number="23" name="tOrigins" color="15" fill="1" visible="yes" active="no"/>
-<layer number="24" name="bOrigins" color="15" fill="1" visible="yes" active="no"/>
-<layer number="25" name="tNames" color="7" fill="1" visible="yes" active="no"/>
-<layer number="26" name="bNames" color="7" fill="1" visible="yes" active="no"/>
-<layer number="27" name="tValues" color="7" fill="1" visible="yes" active="no"/>
-<layer number="28" name="bValues" color="7" fill="1" visible="yes" active="no"/>
+<layer number="1" name="Top" color="4" fill="1" visible="no" active="no"/>
+<layer number="16" name="Bottom" color="1" fill="1" visible="no" active="no"/>
+<layer number="17" name="Pads" color="2" fill="1" visible="no" active="no"/>
+<layer number="18" name="Vias" color="2" fill="1" visible="no" active="no"/>
+<layer number="19" name="Unrouted" color="6" fill="1" visible="no" active="no"/>
+<layer number="20" name="Dimension" color="24" fill="1" visible="no" active="no"/>
+<layer number="21" name="tPlace" color="7" fill="1" visible="no" active="no"/>
+<layer number="22" name="bPlace" color="7" fill="1" visible="no" active="no"/>
+<layer number="23" name="tOrigins" color="15" fill="1" visible="no" active="no"/>
+<layer number="24" name="bOrigins" color="15" fill="1" visible="no" active="no"/>
+<layer number="25" name="tNames" color="7" fill="1" visible="no" active="no"/>
+<layer number="26" name="bNames" color="7" fill="1" visible="no" active="no"/>
+<layer number="27" name="tValues" color="7" fill="1" visible="no" active="no"/>
+<layer number="28" name="bValues" color="7" fill="1" visible="no" active="no"/>
 <layer number="29" name="tStop" color="7" fill="3" visible="no" active="no"/>
 <layer number="30" name="bStop" color="7" fill="6" visible="no" active="no"/>
@@
 <layer number="35" name="tGlue" color="7" fill="4" visible="no" active="no"/>
 <layer number="36" name="bGlue" color="7" fill="5" visible="no" active="no"/>
-<layer number="37" name="tTest" color="7" fill="1" visible="yes" active="no"/>
-<layer number="38" name="bTest" color="7" fill="1" visible="yes" active="no"/>
+<layer number="37" name="tTest" color="7" fill="1" visible="no" active="no"/>
+<layer number="38" name="bTest" color="7" fill="1" visible="no" active="no"/>
 <layer number="39" name="tKeepout" color="4" fill="11" visible="no" active="no"/>
 <layer number="40" name="bKeepout" color="1" fill="11" visible="no" active="no"/>
@@
 <layer number="44" name="Drills" color="7" fill="1" visible="no" active="no"/>
 <layer number="45" name="Holes" color="7" fill="1" visible="no" active="no"/>
-<layer number="46" name="Milling" color="3" fill="1" visible="yes" active="no"/>
-<layer number="47" name="Measures" color="7" fill="1" visible="yes" active="no"/>
-<layer number="48" name="Document" color="7" fill="1" visible="yes" active="no"/>
-<layer number="49" name="Reference" color="7" fill="1" visible="yes" active="no"/>
-<layer number="50" name="dxf" color="7" fill="1" visible="yes" active="no"/>
-<layer number="51" name="tDocu" color="7" fill="1" visible="yes" active="no"/>
-<layer number="52" name="bDocu" color="7" fill="1" visible="yes" active="no"/>
-<layer number="53" name="tGND_GNDA" color="7" fill="9" visible="yes" active="no"/>
-<layer number="54" name="bGND_GNDA" color="1" fill="9" visible="yes" active="no"/>
-<layer number="56" name="wert" color="7" fill="1" visible="yes" active="no"/>
-<layer number="57" name="tCAD" color="7" fill="1" visible="yes" active="no"/>
-<layer number="59" name="tCarbon" color="7" fill="1" visible="yes" active="no"/>
-<layer number="60" name="bCarbon" color="7" fill="1" visible="yes" active="no"/>
+<layer number="46" name="Milling" color="3" fill="1" visible="no" active="no"/>
+<layer number="47" name="Measures" color="7" fill="1" visible="no" active="no"/>
+<layer number="48" name="Document" color="7" fill="1" visible="no" active="no"/>
+<layer number="49" name="Reference" color="7" fill="1" visible="no" active="no"/>
+<layer number="50" name="dxf" color="7" fill="1" visible="no" active="no"/>
+<layer number="51" name="tDocu" color="7" fill="1" visible="no" active="no"/>
+<layer number="52" name="bDocu" color="7" fill="1" visible="no" active="no"/>
+<layer number="53" name="tGND_GNDA" color="7" fill="9" visible="no" active="no"/>
+<layer number="54" name="bGND_GNDA" color="1" fill="9" visible="no" active="no"/>
+<layer number="56" name="wert" color="7" fill="1" visible="no" active="no"/>
+<layer number="57" name="tCAD" color="7" fill="1" visible="no" active="no"/>
+<layer number="59" name="tCarbon" color="7" fill="1" visible="no" active="no"/>
+<layer number="60" name="bCarbon" color="7" fill="1" visible="no" active="no"/>
 <layer number="88" name="SimResults" color="9" fill="1" visible="yes" active="yes"/>
 <layer number="89" name="SimProbes" color="9" fill="1" visible="yes" active="yes"/>
@@
 <part name="C4" library="microbuilder" deviceset="CAP_CERAMIC" device="0805-NOOUTLINE" value="4.7uF"/>
 <part name="C5" library="microbuilder" deviceset="CAP_CERAMIC" device="0805-NOOUTLINE" value="4.7uF"/>
+<part name="IC2" library="linear" library_urn="urn:adsk.eagle:library:262" deviceset="LM2937" device="" package3d_urn="urn:adsk.eagle:package:16425/2"/>
 </parts>
 <sheets>
@@
 <attribute name="NAME" x="178.05" y="-77.49" size="1.27" layer="95" font="vector" rot="R90" align="center"/>
 <attribute name="VALUE" x="182.64" y="-77.49" size="1.27" layer="96" font="vector" rot="R90" align="center"/>
+</instance>
+<instance part="IC2" gate="G$1" x="53.34" y="-27.94" smashed="yes">
+<attribute name="NAME" x="45.72" y="-22.225" size="1.778" layer="95"/>
+<attribute name="VALUE" x="45.72" y="-24.765" size="1.778" layer="96"/>
 </instance>
 </instances>
@@
 <junction x="170.18" y="50.8"/>
 </segment>
-</net>
-<net name="5V" class="0">
-<segment>
-<pinref part="USB_KEYBOARD" gate="G$1" pin="1"/>
-<wire x1="124.46" y1="-119.38" x2="121.92" y2="-119.38" width="0.1524" layer="91"/>
-<label x="121.92" y="-119.38" size="1.778" layer="95"/>
-</segment>
-<segment>
-<pinref part="X2" gate="-39" pin="1"/>
-<wire x1="157.48" y1="-116.84" x2="152.4" y2="-116.84" width="0.1524" layer="91"/>
-<label x="152.4" y="-116.84" size="1.778" layer="95"/>
-</segment>
-<segment>
-<pinref part="X2" gate="-40" pin="1"/>
-<wire x1="157.48" y1="-119.38" x2="152.4" y2="-119.38" width="0.1524" layer="91"/>
-<label x="152.4" y="-119.38" size="1.778" layer="95"/>
-</segment>
-<segment>
-<pinref part="CONNHEADER" gate="G$1" pin="8"/>
-<wire x1="101.6" y1="-55.88" x2="106.68" y2="-55.88" width="0.1524" layer="91"/>
-<label x="101.6" y="-55.88" size="1.778" layer="95"/>
-</segment>
-<segment>
-<pinref part="U2" gate="G$1" pin="VCC"/>
-<wire x1="147.32" y1="63.5" x2="154.94" y2="63.5" width="0.1524" layer="91"/>
-<label x="149.86" y="63.5" size="1.778" layer="95"/>
+<segment>
+<pinref part="IC2" gate="G$1" pin="GND"/>
+<wire x1="53.34" y1="-35.56" x2="53.34" y2="-40.64" width="0.1524" layer="91"/>
+<label x="53.34" y="-40.64" size="1.778" layer="95"/>
 </segment>
 </net>
@@
 <pinref part="C5" gate="G$1" pin="1"/>
 </segment>
+<segment>
+<pinref part="IC2" gate="G$1" pin="VO"/>
+<wire x1="63.5" y1="-27.94" x2="71.12" y2="-27.94" width="0.1524" layer="91"/>
+<label x="66.04" y="-27.94" size="1.778" layer="95"/>
+</segment>
 </net>
 <net name="INT" class="0">
@@
 <label x="195.58" y="25.4" size="1.778" layer="95"/>
 </segment>
-</net>
+<segment>
+<pinref part="IC2" gate="G$1" pin="VI"/>
+<wire x1="35.56" y1="-27.94" x2="43.18" y2="-27.94" width="0.1524" layer="91"/>
+<label x="33.02" y="-27.94" size="1.778" layer="95"/>
+</segment>
+<segment>
+<pinref part="USB_KEYBOARD" gate="G$1" pin="1"/>
+<wire x1="124.46" y1="-119.38" x2="121.92" y2="-119.38" width="0.1524" layer="91"/>
+<label x="121.92" y="-119.38" size="1.778" layer="95"/>
+</segment>
+<segment>
+<pinref part="X2" gate="-39" pin="1"/>
+<wire x1="157.48" y1="-116.84" x2="152.4" y2="-116.84" width="0.1524" layer="91"/>
+<label x="152.4" y="-116.84" size="1.778" layer="95"/>
+</segment>
+<segment>
+<pinref part="X2" gate="-40" pin="1"/>
+<wire x1="157.48" y1="-119.38" x2="152.4" y2="-119.38" width="0.1524" layer="91"/>
+<label x="152.4" y="-119.38" size="1.778" layer="95"/>
+</segment>
+<segment>
+<pinref part="CONNHEADER" gate="G$1" pin="8"/>
+<wire x1="101.6" y1="-55.88" x2="106.68" y2="-55.88" width="0.1524" layer="91"/>
+<label x="101.6" y="-55.88" size="1.778" layer="95"/>
+</segment>
+<segment>
+<pinref part="U2" gate="G$1" pin="VCC"/>
+<wire x1="147.32" y1="63.5" x2="154.94" y2="63.5" width="0.1524" layer="91"/>
+<label x="149.86" y="63.5" size="1.778" layer="95"/>
+</segment>
+</net>

Commit message: .
Parts:
- removed IC2: LM2937, linear:LM2937
- removed U$6: MBT3904DW1T1G, MBT3904DW1T1G:MBT3904DW1T1G
- removed U4: UDA1334ATS, microbuilder:AUDIO_I2S_UDA1334""
- removed USB_KEYBOARD: (no value), con-berg:PN87520
- removed X1: (no value), microbuilder:USB_C
- added J1: CSP-USC16-TR, CSP-USC16-TR:CSP-USC16-TR
- added REG: TS1117BCW33_RPG, TS1117BCW33_RPG:TS1117BCW33_RPG
- added RESET: MBT3904DW1T1G, MBT3904DW1T1G:MBT3904DW1T1G
- added UDA1334: UDA1334ATS, microbuilder:AUDIO_I2S_UDA1334""
- added USBKB: USB-A-S-X-X-SM2, USB-A-S-X-X-SM2:USB-A-S-X-X-SM2
- R1, R10, R11, R12, R13, R14, R15, R16, R17, R18, R5, R6, R7: device microbuilder:RESISTOR_0603_NOOUT -> adafruit:R-US_R0805
- R2, R22, R23, R3, R4, R8, R9: device microbuilder:RESISTOR0805_NOOUTLINE -> adafruit:R-US_R0805
- renumbered IC1 to CP2102, U2 to 6N138, X3 to MIDI_OUT_CONN, X5 to MIDI_IN_CONN, X6 to AUDIO_CONN
Connections:
- removed net CC1: R11.2, X1.CC1
- removed net CC2: R10.2, X1.CC2
- new net N$3: J1.CC2, R11.2
- new net N$4: J1.CC1, R10.2
- net !DTR: now also RESET.4; no longer U$6.4
- net !RTS: now also RESET.1; no longer U$6.1
- net 3V3: now also REG.OUTPUT, UDA1334.VDDD; no longer IC2.VO, U4.VDDD
- net 5V_USB: now also J1.VBUS_A, J1.VBUS_B, REG.INPUT, USBKB.VCC; no longer IC2.VI, USB_KEYBOARD.1, X1.VBUS
- net AGND: now also UDA1334.VSSA; no longer U4.VSSA
- net BCLK: now also UDA1334.BCK; no longer U4.BCK
- net D+: now also USBKB.D+; no longer USB_KEYBOARD.3
- net D-: now also USBKB.D-; no longer USB_KEYBOARD.2
- net DIN: now also UDA1334.DATAI; no longer U4.DATAI
- net ESP32_EN: now also RESET.6; no longer U$6.6
- net GND: now also J1.GND_A, J1.GND_B, J1.SHELL_GND, REG.FIXED/ADJ, UDA1334.DEEM/CLKOUT, UDA1334.MUTE, UDA1334.PLL0, UDA1334.SFOR0, UDA1334.SFOR1, UDA1334.SYSCLK/PLL1, UDA1334.VSSD, USBKB.GND, USBKB.SHIELD; no longer IC2.GND, U4.DEEM/CLKOUT, U4.MUTE, U4.PLL0, U4.SFOR0, U4.SFOR1, U4.SYSCLK/PLL1, U4.VSSD, USB_KEYBOARD.4, X1.GND
- net IO0: now also RESET.3; no longer U$6.3
- net LRC: now also UDA1334.WS; no longer U4.WS
- net N$1: now also RESET.2; no longer U$6.2
- net N$10: now also UDA1334.VREF(DAC); no longer U4.VREF(DAC)
- net N$11: now also UDA1334.VOUTR; no longer U4.VOUTR
- net N$12: now also UDA1334.VOUTL; no longer U4.VOUTL
- net N$2: now also RESET.5; no longer U$6.5
- net N$5: now also UDA1334.VDDA; no longer U4.VDDA
- net USBC_D+: now also J1.DP1; no longer X1.D+
- net USBC_D-: now also J1.DN1; no longer X1.D-
Other:
- note removed: "where does 3v3 come from"
- moved on the sheet: C11, C12, C13, C14, C15, C16, C17, C18, C19, C20, C4, FB3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

Commit message: .
Parts:
- removed 6N138: 6N138SDM, 6N138SDM:6N138SDM
- removed C11, C12, C15: 0.1uF, microbuilder:CAP_CERAMIC0805-NOOUTLINE
- removed C13, C14: 0.01uF, microbuilder:CAP_CERAMIC0805-NOOUTLINE
- removed C16, C17: 47uF, microbuilder:CAP_ELECTROLYTICPANASONIC_C
- removed C18, C19, C20: 10uF, microbuilder:CAP_CERAMIC0805-NOOUTLINE
- removed CP2102: CP2102N-A02-GQFN24, CP2102N-A02-GQFN24:CP2102N-A02-GQFN24
- removed FB3, FB4: Ferrite, microbuilder:FERRITE0805
- removed R22, R8: 220k, adafruit:R-US_R0805
- removed R23, R9: 100, adafruit:R-US_R0805
- removed R4: 10k, adafruit:R-US_R0805
- removed REG: TS1117BCW33_RPG, TS1117BCW33_RPG:TS1117BCW33_RPG
- removed UDA1334: UDA1334ATS, microbuilder:AUDIO_I2S_UDA1334""
- added 6N137S: 6N137S, 6N137S:6N137S
- added C10, C21, C8, C9: 0.1uF, microbuilder:CAP_CERAMIC0805-NOOUTLINE
- added C22, C23: 2.2uF, microbuilder:CAP_CERAMIC0805-NOOUTLINE
- added C28, C29, C30, C31: 10uF, microbuilder:CAP_ELECTROLYTICPANASONIC_C
- added C32, C33: 2.2nF, microbuilder:CAP_CERAMIC0805-NOOUTLINE
- added R19, R20: 470, adafruit:R-US_R0805
- added U2: INTERFACE-CP2102-GMR(QFN28), INTERFACE-CP2102-GMR_QFN28_:INTERFACE-CP2102-GMR(QFN28)
- added U3: PCM5101APW, pcm5101apw:PCM5101APW
Connections:
- removed net N$10: C15.1, C20.1, UDA1334.VREF(DAC)
- removed net N$11: C17.+, UDA1334.VOUTR
- removed net N$12: C16.+, UDA1334.VOUTL
- removed net N$5: C11.1, C18.1, FB3.P$1, UDA1334.VDDA
- removed net N$6: C16.-, R8.2, R9.1
- removed net N$9: C17.-, R22.2, R23.1
- removed net USB_RESET: CP2102.RSTB, R4.1
- new net N$16: C22.1, U3.CAPM
- new net N$18: C22.2, U3.CAPP
- new net N$7: C28.+, C8.1, U3.LDOO
- new net N$8: R19.2, U3.OUTR
- new net OUTL: R20.2, U3.OUTL
- new net VNEG: C23.1, U3.VNEG
- net !DTR: now also U2.DTR; no longer CP2102.DTR
- net !RTS: now also U2.RTS; no longer CP2102.RTS
- net 3V3: now also C10.2, C21.2, C29.+, C30.+, C31.+, C9.2, U2.VDD, U3.AVDD, U3.CPVDD, U3.DVDD, U3.XSMT; no longer C12.1, C19.1, FB3.P$2, REG.OUTPUT, UDA1334.VDDD
- net 3V3_USB: no longer CP2102.VDD, CP2102.VIO, R4.2
- net 5V_USB: now also 6N137S.VCC, U2.REGIN; no longer 6N138.VCC, CP2102.VREGIN, REG.INPUT
- net AGND: now also C21.1, C23.2, C30.-, C31.-, C32.2, C33.2, C9.1, U3.AGND, U3.CPGND; no longer C11.2, C13.2, C14.2, C15.2, C18.2, C20.2, FB4.P$1, R22.1, R8.1, UDA1334.VSSA
- net BCLK: now also U3.BCK; no longer UDA1334.BCK
- net DIN: now also U3.DIN; no longer UDA1334.DATAI
- net GND: now also 6N137S.GND, C10.1, C28.-, C29.-, C8.2, U2.GND, U2.GND@1, U3.DEMP, U3.DGND, U3.FLT, U3.FMT, U3.SCK; no longer 6N138.GND, C12.2, C19.2, CP2102.GND_1, CP2102.GND_2, FB4.P$2, REG.FIXED/ADJ, UDA1334.DEEM/CLKOUT, UDA1334.MUTE, UDA1334.PLL0, UDA1334.SFOR0, UDA1334.SFOR1, UDA1334.SYSCLK/PLL1, UDA1334.VSSD
- net LOUT: now also C33.1, R20.1; no longer C13.1, R9.2
- net LRC: now also U3.LRCK; no longer UDA1334.WS
- net MIDI_IN: now also 6N137S.VOUT; no longer 6N138.VO
- net MIDI_IN_SINK: now also 6N137S.C; no longer 6N138.C
- net N$30: now also 6N137S.A; no longer 6N138.A
- net N$32: now also 6N137S.EN; no longer 6N138.VB
- net ROUT: now also C32.1, R19.1; no longer C14.1, R23.2
- net UART0_RXD: now also U2.TXD; no longer CP2102.TXD
- net UART0_TXD: now also U2.RXD; no longer CP2102.RXD
- net USBC_D+: now also U2.D+; no longer CP2102.D+
- net USBC_D-: now also U2.D-; no longer CP2102.D-
- net USB_VBUS: now also U2.VBUS; no longer CP2102.VBUS
Other:
- moved on the sheet: R16

Commit message: .
Parts:
- added R4: 10k, adafruit:R-US_R0805
Connections:
- removed net 3V3_USB: C2.1, C3.1
- new net USB_RESET: R4.1, U2.!RST
- net 3V3: now also C2.1, C3.1, R4.2
Changed lines of the file:
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@@
 <part name="C32" library="microbuilder" deviceset="CAP_CERAMIC" device="0805-NOOUTLINE" value="2.2nF"/>
 <part name="C33" library="microbuilder" deviceset="CAP_CERAMIC" device="0805-NOOUTLINE" value="2.2nF"/>
+<part name="R4" library="adafruit" deviceset="R-US_" device="R0805" value="10k"/>
 </parts>
 <sheets>
@@
 <attribute name="NAME" x="416.81" y="-156.23" size="1.27" layer="95" font="vector" rot="R90" align="center"/>
 <attribute name="VALUE" x="421.4" y="-156.23" size="1.27" layer="96" font="vector" rot="R90" align="center"/>
+</instance>
+<instance part="R4" gate="G$1" x="307.34" y="12.7" smashed="yes" rot="R90">
+<attribute name="NAME" x="304.8" y="12.7" size="1.27" layer="95" font="vector" rot="R90" align="center"/>
+<attribute name="VALUE" x="307.34" y="12.7" size="1.016" layer="96" font="vector" ratio="15" rot="R90" align="center"/>
 </instance>
 </instances>
@@
 <label x="383.54" y="-190.5" size="1.778" layer="95"/>
 </segment>
+<segment>
+<wire x1="312.42" y1="-5.08" x2="312.42" y2="-7.62" width="0.1524" layer="91"/>
+<label x="309.88" y="-5.08" size="1.778" layer="95"/>
+<pinref part="C2" gate="G$1" pin="1"/>
+<pinref part="C3" gate="G$1" pin="1"/>
+<wire x1="325.12" y1="-7.62" x2="312.42" y2="-7.62" width="0.1524" layer="91"/>
+<junction x="312.42" y="-7.62"/>
+</segment>
+<segment>
+<pinref part="R4" gate="G$1" pin="2"/>
+<wire x1="307.34" y1="20.32" x2="307.34" y2="17.78" width="0.1524" layer="91"/>
+<label x="307.34" y="17.78" size="1.778" layer="95" rot="R90"/>
+</segment>
 </net>
 <net name="INT" class="0">
@@
 </segment>
 </net>
-<net name="3V3_USB" class="0">
-<segment>
-<wire x1="312.42" y1="-5.08" x2="312.42" y2="-7.62" width="0.1524" layer="91"/>
-<label x="309.88" y="-5.08" size="1.778" layer="95"/>
-<pinref part="C2" gate="G$1" pin="1"/>
-<pinref part="C3" gate="G$1" pin="1"/>
-<wire x1="325.12" y1="-7.62" x2="312.42" y2="-7.62" width="0.1524" layer="91"/>
-<junction x="312.42" y="-7.62"/>
-</segment>
-</net>
 <net name="5V_USB" class="0">
 <segment>
@@
 </segment>
 </net>
+<net name="USB_RESET" class="0">
+<segment>
+<pinref part="U2" gate="G$1" pin="!RST"/>
+<wire x1="238.76" y1="88.9" x2="238.76" y2="83.82" width="0.1524" layer="91"/>
+<label x="238.76" y="73.66" size="1.778" layer="95" rot="R90"/>
+</segment>
+<segment>
+<pinref part="R4" gate="G$1" pin="1"/>
+<wire x1="307.34" y1="7.62" x2="307.34" y2="5.08" width="0.1524" layer="91"/>
+<wire x1="307.34" y1="5.08" x2="299.72" y2="5.08" width="0.1524" layer="91"/>
+<label x="292.1" y="5.08" size="1.778" layer="95"/>
+</segment>
+</net>
