File: pcbs/tulip4_board_ch340e_rev2/tulip breakout.sch (EAGLE design)
At the start: 59 parts, among them IC1 MCP73831/OT, J1 CSP-USC16-TR, U1 ESP32-S3-WROOM-2-N32R8V, U2 LD29150DT33R, U3 PCM5101APW, U6 CH340C, X2 FH12-40S-0.5SH

Commit message: .
Parts:
- removed SERIAL: (no value), adafruit:PINHD-1X6
- added BOOST, MCP: (no value), jumper:SJW
- added J2: (no value), SparkFun-Connectors:CONN_10"
Connections:
- new net N$4: IC1.VDD, MCP.2
- new net N$5: BOOST.2, U$22.VIN
- net !DTR: now also J2.3; no longer SERIAL.2
- net !RTS: now also J2.4; no longer SERIAL.6
- net 3V3: now also J2.8
- net 5V: now also J2.9; no longer SERIAL.3
- net 5V_USB: now also J2.7, MCP.1; no longer IC1.VDD
- net DN1: now also J2.1
- net DP1: now also J2.2
- net GND: now also J2.10; no longer SERIAL.1
- net UART0_RXD: now also J2.6; no longer SERIAL.4
- net UART0_TXD: now also J2.5; no longer SERIAL.5
- net VBATT: now also BOOST.1; no longer U$22.VIN
Other:
- moved on the sheet: C14, R23

Commit message: .
Parts:
- removed BOOST: (no value), jumper:SJW
- added BOOST1: (no value), jumper:SJW
Connections:
- removed net N$5: BOOST.2, U$22.VIN
- new net N$6: BOOST1.2, L2.1, R23.1, U$22.VIN
- net VBATT: now also BOOST1.1; no longer BOOST.1, L2.1, R23.1
Other:
- moved on the sheet: C14
Changed lines of the file:
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@@
 <part name="J2" library="SparkFun-Connectors" library_urn="urn:adsk.eagle:library:513" deviceset="CONN_10" device="&quot;" package3d_urn="urn:adsk.eagle:package:38157/1"/>
 <part name="MCP" library="jumper" library_urn="urn:adsk.eagle:library:252" deviceset="SJ" device="W" package3d_urn="urn:adsk.eagle:package:15507/1"/>
-<part name="BOOST" library="jumper" library_urn="urn:adsk.eagle:library:252" deviceset="SJ" device="W" package3d_urn="urn:adsk.eagle:package:15507/1"/>
+<part name="BOOST1" library="jumper" library_urn="urn:adsk.eagle:library:252" deviceset="SJ" device="W" package3d_urn="urn:adsk.eagle:package:15507/1"/>
 </parts>
 <sheets>
@@
 <attribute name="VALUE" x="208.52" y="54.63" size="1.27" layer="96" font="vector" rot="R270" align="center"/>
 </instance>
-<instance part="C14" gate="G$1" x="177.8" y="124.46" smashed="yes" rot="R180">
-<attribute name="NAME" x="180.09" y="123.21" size="1.27" layer="95" font="vector" rot="R270" align="center"/>
-<attribute name="VALUE" x="175.5" y="123.21" size="1.27" layer="96" font="vector" rot="R270" align="center"/>
+<instance part="C14" gate="G$1" x="167.64" y="124.46" smashed="yes" rot="R180">
+<attribute name="NAME" x="169.93" y="123.21" size="1.27" layer="95" font="vector" rot="R270" align="center"/>
+<attribute name="VALUE" x="165.34" y="123.21" size="1.27" layer="96" font="vector" rot="R270" align="center"/>
 </instance>
 <instance part="C15" gate="G$1" x="254" y="121.92" smashed="yes" rot="R180">
@@
 <attribute name="VALUE" x="213.36" y="62.23" size="1.778" layer="96"/>
 </instance>
-<instance part="BOOST" gate="1" x="198.12" y="119.38" smashed="yes">
-<attribute name="NAME" x="195.58" y="121.92" size="1.778" layer="95"/>
-<attribute name="VALUE" x="195.58" y="115.57" size="1.778" layer="96"/>
+<instance part="BOOST1" gate="1" x="180.34" y="127" smashed="yes">
+<attribute name="NAME" x="177.8" y="129.54" size="1.778" layer="95"/>
+<attribute name="VALUE" x="177.8" y="123.19" size="1.778" layer="96"/>
 </instance>
 </instances>
@@
 <segment>
 <pinref part="C14" gate="G$1" pin="1"/>
-<wire x1="177.8" y1="119.38" x2="177.8" y2="114.3" width="0.1524" layer="91"/>
-<label x="175.26" y="114.3" size="1.778" layer="95"/>
+<wire x1="167.64" y1="119.38" x2="167.64" y2="114.3" width="0.1524" layer="91"/>
+<label x="165.1" y="114.3" size="1.778" layer="95"/>
 </segment>
 <segment>
@@
 </segment>
 <segment>
-<pinref part="R23" gate="G$1" pin="1"/>
-<wire x1="185.42" y1="114.3" x2="185.42" y2="119.38" width="0.1524" layer="91"/>
-<wire x1="185.42" y1="119.38" x2="185.42" y2="127" width="0.1524" layer="91"/>
-<wire x1="185.42" y1="127" x2="177.8" y2="127" width="0.1524" layer="91"/>
 <pinref part="C14" gate="G$1" pin="2"/>
-<wire x1="177.8" y1="127" x2="177.8" y2="132.08" width="0.1524" layer="91"/>
-<junction x="177.8" y="127"/>
-<label x="175.26" y="132.08" size="1.778" layer="95"/>
-<wire x1="185.42" y1="127" x2="205.74" y2="127" width="0.1524" layer="91"/>
-<junction x="185.42" y="127"/>
-<pinref part="L2" gate="G$1" pin="1"/>
-<pinref part="BOOST" gate="1" pin="1"/>
-<wire x1="193.04" y1="119.38" x2="185.42" y2="119.38" width="0.1524" layer="91"/>
-<junction x="185.42" y="119.38"/>
+<wire x1="167.64" y1="127" x2="167.64" y2="132.08" width="0.1524" layer="91"/>
+<label x="165.1" y="132.08" size="1.778" layer="95"/>
+<pinref part="BOOST1" gate="1" pin="1"/>
+<wire x1="167.64" y1="127" x2="175.26" y2="127" width="0.1524" layer="91"/>
+<junction x="167.64" y="127"/>
 </segment>
 </net>
@@
 </segment>
 </net>
-<net name="N$5" class="0">
-<segment>
+<net name="N$6" class="0">
+<segment>
+<pinref part="R23" gate="G$1" pin="1"/>
+<wire x1="185.42" y1="114.3" x2="185.42" y2="119.38" width="0.1524" layer="91"/>
 <pinref part="U$22" gate="G$1" pin="VIN"/>
-<pinref part="BOOST" gate="1" pin="2"/>
-</segment>
-</net>
+<wire x1="185.42" y1="119.38" x2="193.04" y2="119.38" width="0.1524" layer="91"/>
+<pinref part="BOOST1" gate="1" pin="2"/>
+<wire x1="193.04" y1="119.38" x2="203.2" y2="119.38" width="0.1524" layer="91"/>
+<wire x1="185.42" y1="127" x2="193.04" y2="127" width="0.1524" layer="91"/>
+<wire x1="193.04" y1="119.38" x2="193.04" y2="127" width="0.1524" layer="91"/>
+<junction x="193.04" y="119.38"/>
+<pinref part="L2" gate="G$1" pin="1"/>
+<wire x1="193.04" y1="127" x2="205.74" y2="127" width="0.1524" layer="91"/>
+<junction x="193.04" y="127"/>
+</segment>
+</net>
