File: pcbs/tulip4_board_v4r6/tulip breakout.brd (EAGLE design)
At the start: 66.2 x 55.6 mm, 47 parts, among them J1 CSP-USC16-TR, J3 TSM-106-02-L-DH-A, U1 ESP32-S3-WROOM-2-N32R8V, U2 LD29150DT33R, U3 PCM5101APW, U6 CH340C, X2 FH12-40S-0.5SH

Commit message: .
Parts:
- C11: value 10nF -> 10uF
- moved RESET 8.71 mm to (25.9, 52.4)
- moved X2 1.00 mm to (41.1, 52.5)
Connections:
- net 3V3: no longer U6.16
- net 5V_USB: now also U6.16
Routing:
- net PWM: track 54.6 -> 125.9 mm, vias 4 -> 2
- net PCLK: track 111.1 -> 43.2 mm, vias 2 -> 4
- net B7: track 38.9 -> 101.8 mm, vias 4 -> 2
- net BLEN: track 83.0 -> 31.9 mm
- net R7: track 36.5 -> 86.2 mm, vias 2 -> 4
- net G6: track 56.0 -> 99.4 mm, vias 2 -> 4
- net G7: track 83.4 -> 48.1 mm
- net D+: track 34.1 -> 64.7 mm, vias 2 -> 0
- net DIN: track 67.2 -> 96.7 mm
- net GND: track 397.5 -> 368.2 mm, vias 9 -> 8
- net IO0: track 16.9 -> 42.8 mm, vias 2 -> 3
- net 3V3: track 191.3 -> 214.9 mm, vias 13 -> 10
- net !DTR: track 40.8 -> 59.4 mm, vias 4 -> 3
- net G5: track 91.4 -> 109.4 mm, vias 2 -> 4
- net VSYNC: track 34.8 -> 50.9 mm, vias 4 -> 2
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