File: pcbs/tulip4_board_v4r6/tulip breakout.sch (EAGLE design)
At the start: 47 parts, among them J1 CSP-USC16-TR, J3 TSM-106-02-L-DH-A, U1 ESP32-S3-WROOM-2-N32R8V, U2 LD29150DT33R, U3 PCM5101APW, U6 CH340C, X2 FH12-40S-0.5SH

Commit message: .
Parts:
- C11: value 10nF -> 10uF
Connections:
- net 3V3: no longer U6.VCC
- net 5V_USB: now also U6.VCC
Changed lines of the file:
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@@
 <part name="R9" library="adafruit" deviceset="R-US_" device="R0805" value="5.1K"/>
 <part name="R10" library="adafruit" deviceset="R-US_" device="R0805" value="5.1K"/>
-<part name="C11" library="microbuilder" deviceset="CAP_CERAMIC" device="0805-NOOUTLINE" value="10nF"/>
+<part name="C11" library="microbuilder" deviceset="CAP_CERAMIC" device="0805-NOOUTLINE" value="10uF"/>
 <part name="POWER" library="500ASSP1SM6QE" deviceset="500ASSP1SM6QE" device=""/>
 <part name="J3" library="TSM-106-02-L-DH-A" deviceset="TSM-106-02-L-DH-A" device=""/>
@@
 </segment>
 <segment>
-<pinref part="U6" gate="U1" pin="VCC"/>
-<wire x1="294.64" y1="22.86" x2="287.02" y2="22.86" width="0.1524" layer="91"/>
-<label x="287.02" y="22.86" size="1.778" layer="95"/>
-</segment>
-<segment>
 <pinref part="J3" gate="G$1" pin="03"/>
 <wire x1="215.9" y1="86.36" x2="210.82" y2="86.36" width="0.1524" layer="91"/>
@@
 <label x="243.84" y="78.74" size="1.778" layer="95"/>
 </segment>
-</net>
+<segment>
+<pinref part="U6" gate="U1" pin="VCC"/>
+<wire x1="294.64" y1="22.86" x2="287.02" y2="22.86" width="0.1524" layer="91"/>
+<label x="287.02" y="22.86" size="1.778" layer="95"/>
+</segment>
+</net>
