File: docs/pcbs/tulip4_board_v4r7/tulip breakout.brd (EAGLE design)
At the start: 66.2 x 55.6 mm, 49 parts, among them J1 CSP-USC16-TR, J2 440055-3, U1 ESP32-S3-WROOM-2-N32R8V, U2 LD29150DT33R, U3 PCM5101APW, U4 VO0601T, U6 CH340C, X2 FH12-40S-0.5SH

Commit message: submitted r7 board
Parts:
- removed JP1: (no value), adafruit:1X03
- removed U$2: SNESCONN, gamepad-conn:SNESCONN
- removed U1: ESP32-S3-WROOM-2-N32R8V, ESP32-S3-WROOM-2-N32R8V:XCVR_ESP32-S3-WROOM-2-N32R8V
- removed U4: VO0601T, VO0601T:SOIC127P610X331-8N
- removed X2: FH12-40S-0.5SH, con-hirose:FH12-40S-0.5SH
- added ESP32S3: ESP32-S3-WROOM-2-N32R8V, ESP32-S3-WROOM-2-N32R8V:XCVR_ESP32-S3-WROOM-2-N32R8V
- added EXP: (no value), adafruit:1X08-BIG
- added J3: 40PINFPC15-1F-REV, adafruit:XF2M-4015-1F-REVERSE
- added OPTO: VO0601T, VO0601T:SOIC127P610X331-8N
- added SELECT: (no value), adafruit:1X03
- added SNES: SNESCONN, gamepad-conn:SNESCONN
- moved R15 5.91 mm to (31.7, 45.5)
- moved C28 2.42 mm to (16.5, 28.3)
- moved C31 2.40 mm to (16.6, 21.8)
- moved H2 2.02 mm to (48.4, 45.0)
- moved D2 1.50 mm to (52.6, 37.8)
- moved RESET 1.33 mm to (25.6, 51.1)
- moved R13 0.50 mm to (26.0, 45.5)
- moved C5 0.40 mm to (31.7, 33.0)
- moved R7 0.36 mm to (31.7, 42.2)
- moved R1 0.36 mm to (26.1, 42.4)
- moved C11 0.30 mm to (31.5, 39.2)
- moved C4 0.22 mm to (31.6, 36.4)
- renumbered J1 to INPUT, J2 to PWR, U2 to REG, U3 to PCM, U6 to SERIAL
Connections:
- removed net N$10: JP1.2, POWER.2
- removed net PWR: U1.17
- new net IO38: ESP32S3.31, EXP.6
- new net IO9: ESP32S3.17, EXP.8
- new net SELECT: POWER.2, SELECT.2
- net 3V3: now also ESP32S3.2, EXP.2, J3.37; no longer U1.2, X2.37
- net 5V: now also EXP.1, J3.39, J3.40, OPTO.8, SNES.5V; no longer U$2.5V, U4.8, X2.39, X2.40
- net 5V_IN: now also SELECT.3; no longer JP1.3
- net 5V_USB: now also SELECT.1; no longer JP1.1
- net B6: now also ESP32S3.20, J3.14; no longer U1.20, X2.14
- net B7: now also ESP32S3.23, J3.13; no longer U1.23, X2.13
- net BCLK: now also ESP32S3.39; no longer U1.39
- net BLEN: now also ESP32S3.32, J3.10; no longer U1.32, X2.10
- net D+: now also ESP32S3.14; no longer U1.14
- net D-: now also ESP32S3.13; no longer U1.13
- net DE: now also ESP32S3.35, J3.7; no longer U1.35, X2.7
- net DIN: now also ESP32S3.38; no longer U1.38
- net ESP32_EN: now also ESP32S3.3; no longer U1.3
- net G5: now also ESP32S3.12, J3.23; no longer U1.12, X2.23
- net G6: now also ESP32S3.15, J3.22; no longer U1.15, X2.22
- net G7: now also ESP32S3.16, J3.21; no longer U1.16, X2.21
- net GND: now also ESP32S3.1, ESP32S3.40, ESP32S3.41_1, ESP32S3.41_2, ESP32S3.41_3, ESP32S3.41_4, ESP32S3.41_5, ESP32S3.41_6, ESP32S3.41_7, ESP32S3.41_8, ESP32S3.41_9, EXP.3, J3.12, J3.15, J3.16, J3.17, J3.18, J3.19, J3.20, J3.24, J3.25, J3.26, J3.27, J3.28, J3.32, J3.33, J3.34, J3.35, J3.36, J3.38, J3.5, OPTO.5, SNES.GND; no longer U$2.GND, U1.1, U1.40, U1.41_1, U1.41_2, U1.41_3, U1.41_4, U1.41_5, U1.41_6, U1.41_7, U1.41_8, U1.41_9, U4.5, X2.12, X2.15, X2.16, X2.17, X2.18, X2.19, X2.20, X2.24, X2.25, X2.26, X2.27, X2.28, X2.32, X2.33, X2.34, X2.35, X2.36, X2.38, X2.5
- net GPIO10: now also ESP32S3.18; no longer U1.18
- net HSYNC: now also ESP32S3.33, J3.9; no longer U1.33, X2.9
- net INT: now also ESP32S3.5, J3.1; no longer U1.5, X2.1
- net IO0: now also ESP32S3.27, EXP.7; no longer U1.27
- net JOY_CLK: now also ESP32S3.21, SNES.CLOCK; no longer U$2.CLOCK, U1.21
- net JOY_D0: now also ESP32S3.26, SNES.D0; no longer U$2.D0, U1.26
- net JOY_LATCH: now also ESP32S3.25, SNES.LATCH; no longer U$2.LATCH, U1.25
- net LRC: now also ESP32S3.4; no longer U1.4
- net MIDI_IN: now also ESP32S3.24, OPTO.6; no longer U1.24, U4.6
- net MIDI_IN_SINK: now also OPTO.3; no longer U4.3
- net MIDI_OUT: now also ESP32S3.19; no longer U1.19
- net N$30: now also OPTO.2; no longer U4.2
- net N$32: now also OPTO.7; no longer U4.7
- net PCLK: now also ESP32S3.22, J3.11; no longer U1.22, X2.11
- net PWM: now also ESP32S3.9, J3.6; no longer U1.9, X2.6
- net R5: now also ESP32S3.6, J3.31; no longer U1.6, X2.31
- net R6: now also ESP32S3.7, J3.30; no longer U1.7, X2.30
- net R7: now also ESP32S3.8, J3.29; no longer U1.8, X2.29
- net SCL: now also ESP32S3.10, EXP.5, J3.3; no longer U1.10, X2.3
- net SDA: now also ESP32S3.11, EXP.4, J3.4; no longer U1.11, X2.4
- net UART0_RXD: now also ESP32S3.36; no longer U1.36
- net UART0_TXD: now also ESP32S3.37; no longer U1.37
- net VSYNC: now also ESP32S3.34, J3.8; no longer U1.34, X2.8
Routing:
- net N$10: track 114.4 -> 0.00 mm, vias 1 -> 0
- net SELECT: track 0.00 -> 75.0 mm, vias 0 -> 4
- net DIN: track 105.2 -> 41.8 mm, vias 2 -> 4
- net IO9: track 0.00 -> 62.4 mm, vias 0 -> 3
- net R7: track 131.4 -> 73.5 mm, vias 1 -> 3
- net SCL: track 50.7 -> 102.6 mm, vias 3 -> 7
- net IO0: track 24.1 -> 75.9 mm, vias 3 -> 6
- net SDA: track 51.7 -> 100.5 mm, vias 3 -> 6
- net IO38: track 0.00 -> 45.1 mm, vias 0 -> 3
- net G5: track 112.2 -> 67.7 mm
- net GND: track 377.6 -> 419.0 mm, vias 8 -> 3
- net G7: track 92.2 -> 55.7 mm, vias 3 -> 1
- net PWM: track 87.6 -> 122.1 mm, vias 5 -> 3
- net 3V3: track 163.9 -> 196.4 mm
- net G6: track 124.6 -> 92.5 mm, vias 3 -> 5
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Other:
- board text added: "RESET"
- board text added: "tulip.computer v4r7"
- board text removed: "tulip.computer v4r6"

Commit message: .
Parts:
- removed SELECT: (no value), adafruit:1X03
- added EXT-USB: (no value), adafruit:1X03
- moved C31 11.2 mm to (5.70, 19.1)
- moved C28 7.91 mm to (14.0, 20.8)
Connections:
- removed net SELECT: POWER.2, SELECT.2
- new net EXT-USB: EXT-USB.2, POWER.2
- net 5V_IN: now also EXT-USB.3; no longer SELECT.3
- net 5V_USB: now also EXT-USB.1; no longer SELECT.1
Routing:
- net EXT-USB: track 0.00 -> 107.7 mm, vias 0 -> 4
- net B6: track 49.7 -> 125.0 mm
- net G7: track 55.7 -> 130.7 mm, vias 1 -> 3
- net SELECT: track 75.0 -> 0.00 mm, vias 4 -> 0
- net G6: track 92.5 -> 129.5 mm, vias 5 -> 3
- net MIDI_IN_SOURCE: track 89.2 -> 59.2 mm
- net MIDI_IN_SINK: track 73.9 -> 45.1 mm, vias 2 -> 4
- net R7: track 73.5 -> 45.3 mm, vias 3 -> 5
- net BCLK: track 89.8 -> 62.0 mm
- net GND: track 419.0 -> 391.6 mm, vias 3 -> 6
- net G5: track 67.7 -> 86.8 mm, vias 3 -> 5
- net DP1: track 55.3 -> 73.4 mm, vias 4 -> 2
- net PCLK: track 86.1 -> 68.4 mm
- net AGND: track 90.4 -> 105.0 mm, vias 2 -> 4
- net ROUT: track 46.3 -> 59.2 mm
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