File: docs/pcbs/tulip4_board_v4r7/tulip breakout.sch (EAGLE design)
At the start: 49 parts, among them J1 CSP-USC16-TR, J2 440055-3, U1 ESP32-S3-WROOM-2-N32R8V, U2 LD29150DT33R, U3 PCM5101APW, U4 VO0601T, U6 CH340C, X2 FH12-40S-0.5SH

Commit message: submitted r7 board
Parts:
- removed X2: FH12-40S-0.5SH, con-hirose:FH12-40S-0.5SH
- added EXP: (no value), adafruit:PINHD-1X8BIG
- added J3: 40PINFPC15-1F-REV, adafruit:40PINFPC15-1F-REV
- renumbered J1 to INPUT, J2 to PWR, JP1 to SELECT, U$2 to SNES, U1 to ESP32S3, U2 to REG, U3 to PCM, U4 to OPTO, U6 to SERIAL
Connections:
- net N$10 renamed SELECT
- removed net PWR: ESP32S3.IO9
- new net IO38: ESP32S3.IO38, EXP.6
- new net IO9: ESP32S3.IO9, EXP.8
- net 3V3: now also EXP.2, J3-37.MS; no longer X2-37.1
- net 5V: now also EXP.1, J3-39.MS, J3-40.MS; no longer X2-39.1, X2-40.1
- net B6: now also J3-14.MS; no longer X2-14.1
- net B7: now also J3-13.MS; no longer X2-13.1
- net BLEN: now also J3-10.MS; no longer X2-10.1
- net DE: now also J3-7.MS; no longer X2-7.1
- net G5: now also J3-23.MS; no longer X2-23.1
- net G6: now also J3-22.MS; no longer X2-22.1
- net G7: now also J3-21.MS; no longer X2-21.1
- net GND: now also EXP.3, J3-12.MS, J3-15.MS, J3-16.MS, J3-17.MS, J3-18.MS, J3-19.MS, J3-20.MS, J3-24.MS, J3-25.MS, J3-26.MS, J3-27.MS, J3-28.MS, J3-32.MS, J3-33.MS, J3-34.MS, J3-35.MS, J3-36.MS, J3-38.MS, J3-5.MS; no longer X2-12.1, X2-15.1, X2-16.1, X2-17.1, X2-18.1, X2-19.1, X2-20.1, X2-24.1, X2-25.1, X2-26.1, X2-27.1, X2-28.1, X2-32.1, X2-33.1, X2-34.1, X2-35.1, X2-36.1, X2-38.1, X2-5.1
- net HSYNC: now also J3-9.MS; no longer X2-9.1
- net INT: now also J3-1.MSV; no longer X2-1.1
- net IO0: now also EXP.7
- net PCLK: now also J3-11.MS; no longer X2-11.1
- net PWM: now also J3-6.MS; no longer X2-6.1
- net R5: now also J3-31.MS; no longer X2-31.1
- net R6: now also J3-30.MS; no longer X2-30.1
- net R7: now also J3-29.MS; no longer X2-29.1
- net SCL: now also EXP.5, J3-3.MS; no longer X2-3.1
- net SDA: now also EXP.4, J3-4.MS; no longer X2-4.1
- net VSYNC: now also J3-8.MS; no longer X2-8.1

Commit message: .
Parts:
- renumbered SELECT to EXT-USB
Connections:
- net SELECT renamed EXT-USB
Changed lines of the file:
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@@
 <part name="H2" library="holes" library_urn="urn:adsk.eagle:library:237" deviceset="MOUNT-HOLE" device="2.8" package3d_urn="urn:adsk.eagle:package:14271/1"/>
 <part name="OPTO" library="VO0601T" deviceset="VO0601T" device=""/>
-<part name="SELECT" library="adafruit" deviceset="PINHD-1X3" device=""/>
+<part name="EXT-USB" library="adafruit" deviceset="PINHD-1X3" device=""/>
 <part name="SNES" library="gamepad-conn" deviceset="SNESCONN" device=""/>
 <part name="PWR" library="440055-3" deviceset="440055-3" device=""/>
@@
 <attribute name="VALUE" x="43.1712" y="88.8692" size="1.78108125" layer="96"/>
 </instance>
-<instance part="SELECT" gate="A" x="172.72" y="53.34" smashed="yes">
+<instance part="EXT-USB" gate="A" x="172.72" y="53.34" smashed="yes">
 <attribute name="NAME" x="166.37" y="59.055" size="1.778" layer="95"/>
 <attribute name="VALUE" x="166.37" y="45.72" size="1.778" layer="96"/>
@@
 </segment>
 <segment>
-<pinref part="SELECT" gate="A" pin="1"/>
+<pinref part="EXT-USB" gate="A" pin="1"/>
 <wire x1="170.18" y1="55.88" x2="180.34" y2="55.88" width="0.1524" layer="91"/>
 <label x="177.8" y="55.88" size="1.778" layer="95"/>
@@
 <net name="5V_IN" class="0">
 <segment>
-<pinref part="SELECT" gate="A" pin="3"/>
+<pinref part="EXT-USB" gate="A" pin="3"/>
 <wire x1="170.18" y1="50.8" x2="180.34" y2="50.8" width="0.1524" layer="91"/>
 <label x="177.8" y="50.8" size="1.778" layer="95"/>
@@
 </segment>
 </net>
-<net name="SELECT" class="0">
+<net name="EXT-USB" class="0">
 <segment>
 <pinref part="POWER" gate="G$1" pin="COM"/>
 <wire x1="210.82" y1="60.96" x2="213.36" y2="60.96" width="0.1524" layer="91"/>
-<pinref part="SELECT" gate="A" pin="2"/>
+<pinref part="EXT-USB" gate="A" pin="2"/>
 <wire x1="170.18" y1="53.34" x2="210.82" y2="53.34" width="0.1524" layer="91"/>
 <wire x1="210.82" y1="53.34" x2="210.82" y2="60.96" width="0.1524" layer="91"/>
