File: docs/pcbs/tulip4_board_v4r8/tulip breakout.brd (EAGLE design)
At the start: 66.2 x 55.6 mm, 50 parts, among them J3 40PINFPC15-1F-REV

Commit message: r8
Parts:
- EXT-USB: value (none) -> EG1224; device adafruit:1X03 -> EG1224:SW_EG1224
- POWER: value 500ASSP1SM6QE -> EG1224; device 500ASSP1SM6QE:SW_500ASSP1SM6QE -> EG1224:SW_EG1224
- moved H2 61.6 mm to (15.7, 21.3)
- moved SNES 47.2 mm to (30.9, 48.2)
- moved EXP 44.6 mm to (37.3, 2.30)
- moved C31 42.6 mm to (46.8, 7.90)
- moved RESET 29.6 mm to (23.0, 21.6), turned to 270 degrees
- moved C23 26.8 mm to (46.7, 17.2)
- moved H1 26.5 mm to (52.4, 45.0)
- moved R13 25.7 mm to (45.9, 31.2)
- moved EXT-USB 24.1 mm to (17.0, 4.10), turned to 180 degrees
- moved C21 23.7 mm to (38.8, 22.7), turned to 90 degrees
- moved C22 22.6 mm to (25.5, 33.6)
- moved C10 21.8 mm to (25.4, 31.1)
- moved C30 19.7 mm to (38.4, 8.70), turned to 270 degrees
- moved C8 19.5 mm to (33.3, 31.3), turned to 180 degrees
- moved R17 19.5 mm to (52.7, 31.1), turned to 90 degrees
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- renumbered INPUT1 to KEYBD
Routing:
- net GND: track 0.00 -> 402.9 mm, vias 0 -> 6
- net 3V3: track 0.00 -> 228.0 mm, vias 0 -> 6
- net 5V: track 0.00 -> 147.7 mm, vias 0 -> 1
- net SDA: track 0.00 -> 131.1 mm, vias 0 -> 2
- net SCL: track 0.00 -> 126.6 mm, vias 0 -> 7
- net 5V_USB: track 0.00 -> 108.6 mm, vias 0 -> 5
- net IO0: track 0.00 -> 97.6 mm, vias 0 -> 4
- net BCLK: track 0.00 -> 85.2 mm, vias 0 -> 4
- net EXT-USB: track 0.00 -> 84.4 mm, vias 0 -> 1
- net DIN: track 0.00 -> 78.4 mm, vias 0 -> 4
- net AGND: track 0.00 -> 77.9 mm, vias 0 -> 2
- net ESP32_EN: track 0.00 -> 76.4 mm, vias 0 -> 6
- net MIDI_IN_SOURCE: track 0.00 -> 72.2 mm, vias 0 -> 2
- net INT: track 0.00 -> 70.9 mm, vias 0 -> 3
- net IO38: track 0.00 -> 68.7 mm, vias 0 -> 1
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- added copper zone on layer 1, net AGND
- added copper zone on layer 1, net GND
- added copper zone on layer 16, net GND
Other:
- board text added: "0"
- board text added: "38"
- board text added: "3v3"
- board text added: "5v"
- board text added: "9"
- board text added: "Gnd"
- board text added: "scl"
- board text added: "sda"
- board text added: "tulip.computer v4r8"
- board text removed: "tulip.computer v4r7"
