File: docs/pcbs/tulip4_board_v4r8/tulip breakout.sch (EAGLE design)
At the start: 50 parts, among them J3 40PINFPC15-1F-REV

Commit message: r8
Parts:
- EXT-USB: value (none) -> EG1224; device adafruit:PINHD-1X3 -> EG1224:EG1224
- POWER: value 500ASSP1SM6QE -> EG1224; device 500ASSP1SM6QE:500ASSP1SM6QE -> EG1224:EG1224
- renumbered INPUT1 to KEYBD
Connections:
- net 5V: now also POWER.1; no longer POWER.NC
- net EXT-USB: now also POWER.2; no longer POWER.COM
Changed lines of the file:
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@@
 <part name="R10" library="adafruit" deviceset="R-US_" device="R0805" value="5.1K"/>
 <part name="C11" library="microbuilder" deviceset="CAP_CERAMIC" device="0805-NOOUTLINE" value="10uF"/>
-<part name="POWER" library="500ASSP1SM6QE" deviceset="500ASSP1SM6QE" device=""/>
 <part name="H1" library="holes" library_urn="urn:adsk.eagle:library:237" deviceset="MOUNT-HOLE" device="2.8" package3d_urn="urn:adsk.eagle:package:14271/1"/>
 <part name="H2" library="holes" library_urn="urn:adsk.eagle:library:237" deviceset="MOUNT-HOLE" device="2.8" package3d_urn="urn:adsk.eagle:package:14271/1"/>
 <part name="OPTO" library="VO0601T" deviceset="VO0601T" device=""/>
-<part name="EXT-USB" library="adafruit" deviceset="PINHD-1X3" device=""/>
 <part name="SNES" library="gamepad-conn" deviceset="SNESCONN" device=""/>
 <part name="PWR" library="440055-3" deviceset="440055-3" device=""/>
 <part name="J3" library="adafruit" deviceset="40PINFPC" device="15-1F-REV"/>
 <part name="EXP" library="adafruit" deviceset="PINHD-1X8" device="BIG"/>
-<part name="INPUT1" library="CSP-USC16-TR" deviceset="CSP-USC16-TR" device=""/>
+<part name="KEYBD" library="CSP-USC16-TR" deviceset="CSP-USC16-TR" device=""/>
+<part name="POWER" library="EG1224" deviceset="EG1224" device=""/>
+<part name="EXT-USB" library="EG1224" deviceset="EG1224" device=""/>
 </parts>
 <sheets>
@@
 <attribute name="VALUE" x="283.23" y="22.62" size="1.27" layer="96" font="vector" rot="R180" align="center"/>
 </instance>
-<instance part="POWER" gate="G$1" x="220.98" y="60.96" smashed="yes">
-<attribute name="NAME" x="218.44" y="66.04" size="1.27" layer="95"/>
-<attribute name="VALUE" x="218.44" y="55.88" size="1.27" layer="96" align="top-left"/>
-</instance>
 <instance part="H1" gate="G$1" x="157.48" y="88.9" smashed="yes">
 <attribute name="NAME" x="159.512" y="89.4842" size="1.778" layer="95"/>
@@
 <attribute name="NAME" x="43.17196875" y="122.7073" size="1.780809375" layer="95"/>
 <attribute name="VALUE" x="43.1712" y="88.8692" size="1.78108125" layer="96"/>
-</instance>
-<instance part="EXT-USB" gate="A" x="172.72" y="53.34" smashed="yes">
-<attribute name="NAME" x="166.37" y="59.055" size="1.778" layer="95"/>
-<attribute name="VALUE" x="166.37" y="45.72" size="1.778" layer="96"/>
 </instance>
 <instance part="SNES" gate="G$1" x="185.42" y="109.22" smashed="yes"/>
@@
 <attribute name="VALUE" x="217.17" y="-139.7" size="1.778" layer="96"/>
 </instance>
-<instance part="INPUT1" gate="G$1" x="264.16" y="48.26" smashed="yes">
+<instance part="KEYBD" gate="G$1" x="264.16" y="48.26" smashed="yes">
 <attribute name="NAME" x="251.46" y="61.722" size="1.778" layer="95"/>
 <attribute name="VALUE" x="251.46" y="37.338" size="1.778" layer="96" rot="MR180"/>
+</instance>
+<instance part="POWER" gate="G$1" x="243.84" y="91.44" smashed="yes">
+<attribute name="NAME" x="238.76" y="100.33" size="1.27" layer="95"/>
+<attribute name="VALUE" x="238.76" y="82.55" size="1.27" layer="96" align="top-left"/>
+</instance>
+<instance part="EXT-USB" gate="G$1" x="177.8" y="35.56" smashed="yes">
+<attribute name="NAME" x="172.72" y="44.45" size="1.27" layer="95"/>
+<attribute name="VALUE" x="172.72" y="26.67" size="1.27" layer="96" align="top-left"/>
 </instance>
 </instances>
@@
 </segment>
 <segment>
-<pinref part="INPUT1" gate="G$1" pin="GND_A"/>
+<pinref part="KEYBD" gate="G$1" pin="GND_A"/>
 <wire x1="246.38" y1="45.72" x2="236.22" y2="45.72" width="0.1524" layer="91"/>
 <label x="238.76" y="45.72" size="1.778" layer="95"/>
 </segment>
 <segment>
-<pinref part="INPUT1" gate="G$1" pin="GND_B"/>
+<pinref part="KEYBD" gate="G$1" pin="GND_B"/>
 <wire x1="281.94" y1="45.72" x2="292.1" y2="45.72" width="0.1524" layer="91"/>
 <label x="287.02" y="45.72" size="1.778" layer="95"/>
 </segment>
 <segment>
-<pinref part="INPUT1" gate="G$1" pin="SHELL_GND"/>
+<pinref part="KEYBD" gate="G$1" pin="SHELL_GND"/>
 <wire x1="281.94" y1="40.64" x2="292.1" y2="40.64" width="0.1524" layer="91"/>
 <label x="287.02" y="40.64" size="1.778" layer="95"/>
@@
 </segment>
 <segment>
-<pinref part="INPUT1" gate="G$1" pin="DP1"/>
+<pinref part="KEYBD" gate="G$1" pin="DP1"/>
 <wire x1="246.38" y1="53.34" x2="236.22" y2="53.34" width="0.1524" layer="91"/>
 <label x="238.76" y="53.34" size="1.778" layer="95"/>
 </segment>
 <segment>
-<pinref part="INPUT1" gate="G$1" pin="DP2"/>
+<pinref part="KEYBD" gate="G$1" pin="DP2"/>
 <wire x1="281.94" y1="50.8" x2="292.1" y2="50.8" width="0.1524" layer="91"/>
 <label x="287.02" y="50.8" size="1.778" layer="95"/>
@@
 </segment>
 <segment>
-<pinref part="INPUT1" gate="G$1" pin="DN1"/>
+<pinref part="KEYBD" gate="G$1" pin="DN1"/>
 <wire x1="246.38" y1="50.8" x2="236.22" y2="50.8" width="0.1524" layer="91"/>
 <label x="238.76" y="50.8" size="1.778" layer="95"/>
 </segment>
 <segment>
-<pinref part="INPUT1" gate="G$1" pin="DN2"/>
+<pinref part="KEYBD" gate="G$1" pin="DN2"/>
 <wire x1="281.94" y1="53.34" x2="292.1" y2="53.34" width="0.1524" layer="91"/>
 <label x="287.02" y="53.34" size="1.778" layer="95"/>
@@
 </segment>
 <segment>
-<pinref part="EXT-USB" gate="A" pin="1"/>
-<wire x1="170.18" y1="55.88" x2="180.34" y2="55.88" width="0.1524" layer="91"/>
-<label x="177.8" y="55.88" size="1.778" layer="95"/>
-</segment>
-<segment>
 <pinref part="PWR" gate="G$1" pin="2"/>
 <wire x1="114.3" y1="17.78" x2="106.68" y2="17.78" width="0.1524" layer="91"/>
 <label x="106.68" y="17.78" size="1.778" layer="95"/>
+</segment>
+<segment>
+<pinref part="EXT-USB" gate="G$1" pin="1"/>
+<wire x1="187.96" y1="40.64" x2="200.66" y2="40.64" width="0.1524" layer="91"/>
+<label x="193.04" y="40.64" size="1.778" layer="95"/>
 </segment>
 </net>
@@
 </segment>
 <segment>
-<pinref part="POWER" gate="G$1" pin="NC"/>
-<wire x1="228.6" y1="63.5" x2="233.68" y2="63.5" width="0.1524" layer="91"/>
-<label x="231.14" y="63.5" size="1.778" layer="95"/>
-</segment>
-<segment>
 <pinref part="OPTO" gate="G$1" pin="VCC"/>
 <wire x1="63.5" y1="119.38" x2="68.58" y2="119.38" width="0.1524" layer="91"/>
@@
 </segment>
 <segment>
-<pinref part="INPUT1" gate="G$1" pin="VBUS_A"/>
+<pinref part="KEYBD" gate="G$1" pin="VBUS_A"/>
 <wire x1="246.38" y1="58.42" x2="236.22" y2="58.42" width="0.1524" layer="91"/>
 <label x="238.76" y="58.42" size="1.778" layer="95"/>
 </segment>
 <segment>
-<pinref part="INPUT1" gate="G$1" pin="VBUS_B"/>
+<pinref part="KEYBD" gate="G$1" pin="VBUS_B"/>
 <wire x1="281.94" y1="58.42" x2="292.1" y2="58.42" width="0.1524" layer="91"/>
 <label x="287.02" y="58.42" size="1.778" layer="95"/>
 </segment>
+<segment>
+<pinref part="POWER" gate="G$1" pin="1"/>
+<wire x1="254" y1="96.52" x2="261.62" y2="96.52" width="0.1524" layer="91"/>
+<label x="256.54" y="96.52" size="1.778" layer="95"/>
+</segment>
 </net>
 <net name="5V_IN" class="0">
-<segment>
-<pinref part="EXT-USB" gate="A" pin="3"/>
-<wire x1="170.18" y1="50.8" x2="180.34" y2="50.8" width="0.1524" layer="91"/>
-<label x="177.8" y="50.8" size="1.778" layer="95"/>
-</segment>
 <segment>
 <pinref part="PWR" gate="G$1" pin="3"/>
@@
 <label x="106.68" y="15.24" size="1.778" layer="95"/>
 </segment>
+<segment>
+<pinref part="EXT-USB" gate="G$1" pin="3"/>
+<wire x1="187.96" y1="35.56" x2="200.66" y2="35.56" width="0.1524" layer="91"/>
+<label x="193.04" y="35.56" size="1.778" layer="95"/>
+</segment>
 </net>
 <net name="EXT-USB" class="0">
 <segment>
-<pinref part="POWER" gate="G$1" pin="COM"/>
-<wire x1="210.82" y1="60.96" x2="213.36" y2="60.96" width="0.1524" layer="91"/>
-<pinref part="EXT-USB" gate="A" pin="2"/>
-<wire x1="170.18" y1="53.34" x2="210.82" y2="53.34" width="0.1524" layer="91"/>
-<wire x1="210.82" y1="53.34" x2="210.82" y2="60.96" width="0.1524" layer="91"/>
-</segment>
-</net>
+<pinref part="POWER" gate="G$1" pin="2"/>
+<wire x1="210.82" y1="53.34" x2="210.82" y2="93.98" width="0.1524" layer="91"/>
+<wire x1="210.82" y1="93.98" x2="233.68" y2="93.98" width="0.1524" layer="91"/>
+<pinref part="EXT-USB" gate="G$1" pin="2"/>
+<wire x1="210.82" y1="53.34" x2="167.64" y2="53.34" width="0.1524" layer="91"/>
+<wire x1="167.64" y1="53.34" x2="167.64" y2="38.1" width="0.1524" layer="91"/>
+</segment>
+</net>
