File: docs/pcbs/tulip5_board_v4r9/tulipcc.kicad_sch (KiCad schematic)
At the start: 0 parts

Commit message: Renaming V5R0 to V4R9
Other:
- title: Tulip Creative Computer V5 R0 -> Tulip Creative Computer V4 R9
Changed lines of the file:
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@@
   (paper "A4")
   (title_block
-    (title "Tulip Creative Computer V5 R0")
+    (title "Tulip Creative Computer V4 R9")
   )
   (rectangle (start 52.07 106.68) (end 92.71 130.81)
