File: docs/pcbs/tulip4_board_v4r9/mcu.kicad_sch (KiCad schematic)
At the start: 9 parts, among them U1 ESP32-S3-WROOM-2-N32R8V, U6 MBT3904DW1T1G

Commit message: Progress routing
Parts:
- added C?: 0.1uF, tulipcc_footprint_lib:C_0805_2012, symbol tulipcc_symbol_lib:CAP_0805_0.1UF
- added C?: 22uF, tulipcc_footprint_lib:C_1210_3225, symbol tulipcc_symbol_lib:CAP_1210_22UF
- renumbered C24 to C?, R14 to R?, R11 to R?, R12 to R?, R13 to R?, U1 to U?, U6 to U?
Connections:
- net +3.3V: now also C?.1, C?.2
- net GND: now also C?.1, C?.2
Other:
- moved on the sheet: C?, R3, R4, R?, U?
