File: docs/pcbs/tulip4_board_v4r9/power.kicad_sch (KiCad schematic)
At the start: 29 parts, among them J8 1734827-2, Q1 DMP3099L, SW1 JS102011JAQN, U10 MCP73832, U11 MAX17048G, U12 TPS7A4533DCQR, U13 MIC2875-5.0YMT

Commit message: Progress routing
Parts:
- renumbered C27 to C29, C29 to C31, C30 to C32, C31 to C33, C32 to C34, C33 to C35, C34 to C36, C21 to C?
