File: docs/pcbs/amyboard/amyboard.brd (EAGLE design)
At the start: 106 x 48 mm, 155 parts, among them Q1 AO3407, Q2 S8050, Q5 S8050, U1 PCM9211PT, U15 H11L1SR2M, U16 SPX3819, U2 ESP32­S2­SOLO, U3 HX3608, U4 TL074CD, U6 HX3608, U7 GP8413, Y1 22.5792MHZ

Commit message: newest amyboard sch
Parts:
- C12, C14, C16, C2, C3, C42, C43, C44, C45, C8: value 10uF -> 10uF/10V/TAN; device A9G:DISCRETE_C0603 -> rcl:SMC_Z
- C22: value 1uF -> 10uF/10V/TAN; device A9G:DISCRETE_C0402 -> rcl:SMC_Z
- moved C45 32.4 mm to (48.7, 11.9)
- moved C16 28.9 mm to (20.9, 11.2)
- moved CV_OUT1 24.0 mm to (9.50, 42.7)
- moved CV_OUT2 24.0 mm to (20.5, 42.7)
- moved C22 22.7 mm to (50.7, 11.9)
- moved MIDI_IN 22.0 mm to (31.5, 33.0)
- moved SPDIF_IN 22.0 mm to (42.5, 33.0)
- moved R8 21.2 mm to (1.63, 23.7)
- moved C15 20.5 mm to (36.7, 14.5)
- moved R5 20.4 mm to (2.06, 25.3), turned to 90 degrees
- moved R21 20.1 mm to (1.63, 21.6), turned to 0 degrees
- moved C10 19.2 mm to (1.63, 22.7)
- moved R38 18.3 mm to (3.66, 26.2), turned to 180 degrees
- moved C9 18.2 mm to (1.63, 20.5), turned to 180 degrees
- moved R35 16.2 mm to (3.66, 25.1), turned to 0 degrees
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Connections:
- net +3V3: now also C12.+, C14.+, C22.+, C3.+, C45.+; no longer C14.2, C16.2, C43.1, C44.1, C45.1
- net 5V: now also C16.+; no longer C12.2
- net AGND: now also C12.-, C16.-, C22.-, C45.-, C8.-; no longer C12.1, C16.1, C44.2, C45.2, C8.1
- net GND: now also C14.-, C2.-, C3.-, C42.-; no longer C14.1, C22.1, C42.1, C43.2
- net LINX: now also C43.+; no longer C2.1
- net N$22: now also C42.+; no longer C22.2
- net N$4: now also C43.-; no longer C2.2
- net N$48: now also C2.+; no longer C42.2
- net N$5: now also C44.-; no longer C3.2
- net N$6: now also C8.+; no longer C8.2
- net RINX: now also C44.+; no longer C3.1
Routing:
- net +3V3: track 0.00 -> 207.4 mm, vias 0 -> 10
- net AGND: track 0.00 -> 115.6 mm, vias 0 -> 5
- net I2C_SCL: track 0.00 -> 103.5 mm, vias 0 -> 4
- net I2C_SDA: track 0.00 -> 102.7 mm, vias 0 -> 4
- net ADC1: track 0.00 -> 99.6 mm, vias 0 -> 2
- net ADC2: track 0.00 -> 97.0 mm, vias 0 -> 2
- net MIDI_IN: track 0.00 -> 89.3 mm, vias 0 -> 2
- net LRC: track 0.00 -> 85.6 mm, vias 0 -> 2
- net N$58: track 0.00 -> 82.7 mm, vias 0 -> 1
- net AMYOUT: track 0.00 -> 71.8 mm, vias 0 -> 3
- net MPIO: track 0.00 -> 71.0 mm, vias 0 -> 2
- net SPDIFOUT_SIGNAL: track 0.00 -> 71.0 mm, vias 0 -> 3
- net MCLK: track 0.00 -> 68.3 mm, vias 0 -> 2
- net 5V: track 0.00 -> 66.2 mm, vias 0 -> 3
- net BCLK: track 0.00 -> 65.6 mm, vias 0 -> 2
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Other:
- outline, holes or cut-outs redrawn
- board text added: "+"
- board text added: "AmyBoard"
- board text added: "CVIN/"
- board text added: "LINEIN/"
- board text added: "MIDIIN/"
- board text added: "OUT"
- board text added: "OUT1"
- board text added: "OUT2"
- board text added: "SPDIFIN/"
- board text added: "V1.0"
