File: docs/pcbs/amyboard/amyboard.sch (EAGLE design)
At the start: 161 parts, among them Q1 AO3407, Q2 S8050, Q5 S8050, U1 PCM9211PT, U15 H11L1SR2M, U16 SPX3819, U2 ESP32­S2­SOLO, U3 HX3608, U4 TL074CD, U6 HX3608, U7 GP8413, Y1 22.5792MHZ

Commit message: newest amyboard sch
Parts:
- C12, C14, C16, C2, C3, C42, C43, C44, C45, C8: value 10uF -> 10uF/10V/TAN; device A9G:DISCRETE_C-0603 -> rcl:CPOL-USSMCZ
- C22: value 1uF -> 10uF/10V/TAN; device A9G:DISCRETE_C-0402 -> rcl:CPOL-USSMCZ
Connections:
- net +3V3: now also C12.+, C14.+, C22.+, C3.+, C45.+; no longer C14.2, C16.2, C43.1, C44.1, C45.1
- net 5V: now also C16.+; no longer C12.2
- net AGND: now also C12.-, C16.-, C22.-, C45.-, C8.-; no longer C12.1, C16.1, C44.2, C45.2, C8.1
- net GND: now also C14.-, C2.-, C3.-, C42.-; no longer C14.1, C22.1, C42.1, C43.2
- net LINX: now also C43.+; no longer C2.1
- net N$22: now also C42.+; no longer C22.2
- net N$4: now also C43.-; no longer C2.2
- net N$48: now also C2.+; no longer C42.2
- net N$5: now also C44.-; no longer C3.2
- net N$6: now also C8.+; no longer C8.2
- net RINX: now also C44.+; no longer C3.1
Other:
- note added: "Place C20 and C25 close to U4 (TL074)"
- note removed: "Place C20 and C28 close to U4 (TL074)"
